File: KicadJE_AteOhAte/KicadJE_AteOhAte2.sch (KiCad schematic (older format))
At the start: 88 parts, among them J201 In_Accent, J202 In Gate, J203 Out Tom, P201 Doepfer_Power_10pin, Q201 MMBT2222A, Q202 MMBT2222A, Q203 MMBT2222A, Q204 MMBT2907A, Q205 MMBT2222A, Q206 MMBT2222A, SW201 Con/Tom, U201 TL072, U202 TL072

Commit message: Noise added
Parts:
- added C212: 47n, Capacitor_SMD:C_0805_2012Metric_Pad1.15x1.40mm_HandSolder, symbol Device:C
- added C?: 22u, Capacitor_SMD:C_0805_2012Metric_Pad1.15x1.40mm_HandSolder, symbol Device:C
- added C?: 1u, Capacitor_SMD:C_0805_2012Metric_Pad1.15x1.40mm_HandSolder, symbol Device:C
- added C?: 39n, Capacitor_SMD:C_0805_2012Metric_Pad1.15x1.40mm_HandSolder, symbol Device:C
- added C?: 18n, Capacitor_SMD:C_0805_2012Metric_Pad1.15x1.40mm_HandSolder, symbol Device:C
- added JP?: Jumper, Connector_PinHeader_2.54mm:PinHeader_1x02_P2.54mm_Vertical, symbol Device:Jumper
- added Q?: MMBT2222A, Package_TO_SOT_SMD:SOT-23_Handsoldering, symbol MMBT2222A:MMBT2222A
- added R235: 3k3, Resistor_SMD:R_0805_2012Metric_Pad1.15x1.40mm_HandSolder, symbol Device:R
- added R236: 33k, Resistor_SMD:R_0805_2012Metric_Pad1.15x1.40mm_HandSolder, symbol Device:R
- added R?: 100R, Resistor_SMD:R_0805_2012Metric_Pad1.15x1.40mm_HandSolder, symbol Device:R
- added R? (x2): 1M, Resistor_SMD:R_0805_2012Metric_Pad1.15x1.40mm_HandSolder, symbol Device:R
- added R?: 300R, Resistor_SMD:R_0805_2012Metric_Pad1.15x1.40mm_HandSolder, symbol Device:R
- added R?: 330K, Resistor_SMD:R_0805_2012Metric_Pad1.15x1.40mm_HandSolder, symbol Device:R
- added R?: 4k7, Resistor_SMD:R_0805_2012Metric_Pad1.15x1.40mm_HandSolder, symbol Device:R
- added R? (x2): 22k, Resistor_SMD:R_0805_2012Metric_Pad1.15x1.40mm_HandSolder, symbol Device:R
- added RV?: 100K, Potentiometer_THT:Potentiometer_Bourns_3296W_Vertical, symbol Device:R_POT_TRIM
- added RV?: 50K, Potentiometer_THT:Potentiometer_Bourns_3296W_Vertical, symbol Device:R_POT_TRIM
- added U201: TL072, AJ-Dropbox-Kicad:AJ_SO-8_5.3x6.2mm_P1.27mm, symbol Amplifier_Operational:TL072
- Q204: symbol MMBT2907A:MMBT2907A -> MMBT2907_:MMBT2907*
- renumbered C214 to C213, C212 to C214, C213 to C215, D202 to D201, D204 to D202, D201 to D203, D203 to D204, D206 to D205, D205 to D206, R211 to R210, R212 to R211, R216 to R212, R217 to R213, R210 to R214, R213 to R215, R214 to R216, R215 to R217, R222 to R218, R223 to R219, R224 to R220, R227 to R221, R218 to R222, R219 to R223, R221 to R224, R220 to R225, R225 to R226, R226 to R227, R229 to R228, R228 to R229, R231 to R230, R232 to R231, R234 to R232, R235 to R233, R230 to R234, R233 to R237, R239 to R238, R240 to R239, R236 to R240, R237 to R241, R238 to R242, R241 to R243, R242 to R244, R243 to R245, R244 to R246, RV203 to RV202, RV202 to RV203, U201 to U202, U202 to U203
Connections:
- net +12V: now also R?.1, U201.4 (V-)
- net -12V: now also U201.8 (V+)
- net GND: now also R229.2, C?.2, C?.2, Q?.1 (B), R235.1, R?.1, R?.2; no longer R229.1
- net at Q203.1 (B), R232.2: now also R229.1; no longer R229.2
- net PNP_E: now reaches Q201.2 (E), R220.2, R221.2
- net PNP_E: now also Q204.2 (E); no longer Q204.E
- net PNP_B: now reaches R221.1, R228.2
- net PNP_B: now also Q204.1 (B); no longer Q204.B
- net Coupling: now reaches C210.2, R230.2, R231.2
- net Coupling: now also Q204.3 (C); no longer Q204.C
- net at R240.2, R241.1: now also C212.2
- new net: C212.1, R235.2, R236.1
- new net: R?.2, U201.2 (-)
- new net: C?.1, R?.1, U201.3 (+)
- new net: C?.1, R?.2, U201.5 (+)
- new net: C?.1, R?.2, R?.2
- new net: C?.2, Q?.2 (E), R?.1
- new net: R?.1, R?.2, RV?.1
- new net: R?.2, RV?.2
- new net: C?.2, R?.1, R?.2
- new net: JP?.1, RV?.2
- new net NoiseIn: JP?.2, R236.2
- new net PinkNoise: C?.1, RV?.3, U201.6 (-), U201.7
- new net WhiteNoise: R?.1, R?.1, RV?.1, U201.1
Other:
- note added: "Trim for 130mV RMS"
- moved on the sheet: C201, C202, C203, C204, C205, C206, C207, C208, C209, C210, C211, C213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
