File: KicadJE_AteOhAte/_autosave-KicadJE_AteOhAte.kicad_pcb (KiCad board)
At the start: 2 copper layers, 100 x 100 mm, 156 parts, among them J201 In_Accent, J202 In Gate, J203 Out Tom, J301 Out 1, J302 In_1, J303 Out 2, J304 In 2, J305 Out 1 Final, J306 Out 2 Final, P201 Doepfer_Power_10pin, Q201 MMBT2222A, Q202 MMBT2222A, Q203 MMBT2222A, Q204 MMBT2907A, Q205 MMBT2222A, Q206 MMBT2222A, SW201 Con/Tom, U201 TL072, U202 TL072, U301 TL072, U302 TL072

Commit message: Noise added
Parts:
- C202, R201, R202, R203, R204, R205: moved to B.Cu
- J202: footprint Connector_Audio:Jack_3.5mm_Ledino_KB3SPRS_Horizontal -> AJ-Dropbox-Kicad:PJ301SM
- moved R201 163.2 mm to (57.2, 133.7)
- moved R202 158.3 mm to (52.8, 133.7)
- moved J202 153.0 mm to (73.5, 142.1)
- moved C202 152.0 mm to (79.1, 153.3)
- moved R203 140.8 mm to (71.5, 133.7)
- moved R205 135.7 mm to (75.7, 133.7)
- moved J203 118.3 mm to (83.5, 142.1)
- moved R204 117.0 mm to (84.6, 133.7)
- moved SW201 3.21 mm to (82.0, 120.0)

Commit message: Update _autosave-KicadJE_AteOhAte.kicad_pcb
Parts:
- added C205: 39n, Capacitor_SMD:C_0805_2012Metric_Pad1.15x1.40mm_HandSolder, B.Cu at (-10.0, 26.0)
- added C206: 1u, Capacitor_SMD:C_0805_2012Metric_Pad1.15x1.40mm_HandSolder, B.Cu at (-14.8, 28.9)
- added C207: 22u, Capacitor_SMD:C_0805_2012Metric_Pad1.15x1.40mm_HandSolder, B.Cu at (-14.8, 26.0)
- added C208: 18n, Capacitor_SMD:C_0805_2012Metric_Pad1.15x1.40mm_HandSolder, B.Cu at (-20.8, 21.2)
- added C216: 47n, Capacitor_SMD:C_0805_2012Metric_Pad1.15x1.40mm_HandSolder, B.Cu at (-10.0, 28.9)
- added JP201: Jumper, Connector_PinHeader_2.54mm:PinHeader_1x02_P2.54mm_Vertical, F.Cu at (-44.0, 14.0)
- added Q201: MMBT2222A, Package_TO_SOT_SMD:SOT-23_Handsoldering, B.Cu at (-35.8, 15.2)
- added R201: 1M, Resistor_SMD:R_0805_2012Metric_Pad1.15x1.40mm_HandSolder, B.Cu at (-20.8, 18.2)
- added R202: 4k7, Resistor_SMD:R_0805_2012Metric_Pad1.15x1.40mm_HandSolder, B.Cu at (-25.4, 14.0)
- added R203: 330K, Resistor_SMD:R_0805_2012Metric_Pad1.15x1.40mm_HandSolder, B.Cu at (-14.8, 23.1)
- added R204: 100R, Resistor_SMD:R_0805_2012Metric_Pad1.15x1.40mm_HandSolder, B.Cu at (-30.2, 14.0)
- added R205: 22k, Resistor_SMD:R_0805_2012Metric_Pad1.15x1.40mm_HandSolder, B.Cu at (-16.1, 20.1)
- added R206: 1M, Resistor_SMD:R_0805_2012Metric_Pad1.15x1.40mm_HandSolder, B.Cu at (-20.7, 15.3)
- added R207: 22k, Resistor_SMD:R_0805_2012Metric_Pad1.15x1.40mm_HandSolder, B.Cu at (-10.0, 23.1)
- added R208: 300R, Resistor_SMD:R_0805_2012Metric_Pad1.15x1.40mm_HandSolder, B.Cu at (-11.3, 20.1)
- added R243: 3k3, Resistor_SMD:R_0805_2012Metric_Pad1.15x1.40mm_HandSolder, B.Cu at (-15.9, 17.1)
- added R244: 33k, Resistor_SMD:R_0805_2012Metric_Pad1.15x1.40mm_HandSolder, B.Cu at (-15.9, 14.2)
- added RV201: 100K, Potentiometer_THT:Potentiometer_Bourns_3296W_Vertical, F.Cu at (-42.9, 31.2)
- added RV202: 50K, Potentiometer_THT:Potentiometer_Bourns_3296W_Vertical, F.Cu at (-42.9, 24.8)
- added U201: TL072, AJ-Dropbox-Kicad:AJ_SO-8_5.3x6.2mm_P1.27mm, B.Cu at (-22.5, 26.6)
- C201, C203, C204, D207, D208, D209: moved to B.Cu
- C209: renamed from C205; moved to B.Cu
- C210: renamed from C206; moved to B.Cu
- C211: renamed from C207; moved to B.Cu
- C212: renamed from C208; moved to B.Cu
- C213: renamed from C209; moved to B.Cu
- C214: renamed from C210; moved to B.Cu
- C215: renamed from C211; moved to B.Cu
- C217: renamed from C214; moved to B.Cu
- C218: renamed from C212; moved to B.Cu
- C219: renamed from C213; moved to B.Cu
- D201: renamed from D202; moved to B.Cu
- D202: renamed from D204; moved to B.Cu
- D203: renamed from D201; moved to B.Cu
- D204: renamed from D203; moved to B.Cu
- D205: renamed from D206; moved to B.Cu
- D206: renamed from D205; moved to B.Cu
- Q202: renamed from Q201; moved to B.Cu
- Q203: renamed from Q202; moved to B.Cu
- Q204: renamed from Q203; moved to B.Cu
- Q205: renamed from Q204; moved to B.Cu
- Q206: renamed from Q205; moved to B.Cu
- Q207: renamed from Q206; moved to B.Cu
- R214: renamed from R206; moved to B.Cu
- R215: renamed from R207; moved to B.Cu
- R216: renamed from R208; moved to B.Cu
- R217: renamed from R209; moved to B.Cu
- R218: renamed from R211; moved to B.Cu
- R219: renamed from R212; moved to B.Cu
- R220: renamed from R216; moved to B.Cu
- R221: renamed from R217; moved to B.Cu
- R222: renamed from R210; moved to B.Cu
- R223: renamed from R213; moved to B.Cu
- R224: renamed from R214; moved to B.Cu
- R225: renamed from R215; moved to B.Cu
- R226: renamed from R222; moved to B.Cu
- R227: renamed from R223; moved to B.Cu
- R228: renamed from R224; moved to B.Cu
- R229: renamed from R227; moved to B.Cu
- R230: renamed from R218; moved to B.Cu
- R231: renamed from R219; moved to B.Cu
- R232: renamed from R221; moved to B.Cu
- R233: renamed from R220; moved to B.Cu
- R234: renamed from R225; moved to B.Cu
- R235: renamed from R226; moved to B.Cu
- R236: renamed from R229; moved to B.Cu
- R237: renamed from R228; moved to B.Cu
- R238: renamed from R231; moved to B.Cu
- R239: renamed from R232; moved to B.Cu
- R240: renamed from R234; moved to B.Cu
- R241: renamed from R235; moved to B.Cu
- R242: renamed from R230; moved to B.Cu
- R245: renamed from R233; moved to B.Cu
- R246: renamed from R239; moved to B.Cu
- R247: renamed from R240; moved to B.Cu
- R248: renamed from R236; moved to B.Cu
- R249: renamed from R237; moved to B.Cu
- R250: renamed from R238; moved to B.Cu
- R251: renamed from R241; moved to B.Cu
- R252: renamed from R242; moved to B.Cu
- R253: renamed from R243; moved to B.Cu
- R254: renamed from R244; moved to B.Cu
- U202: renamed from U201; moved to B.Cu
- U203: renamed from U202; moved to B.Cu
- moved C202 153.7 mm to (52.0, 2.00)
- moved Q205 116.9 mm to (53.0, 21.0)
- moved R216 68.5 mm to (6.98, 5.37)
- moved R249 68.5 mm to (11.7, 5.37)
- moved R225 67.7 mm to (21.2, 5.77)
- moved R242 67.7 mm to (16.5, 5.77)
- moved C214 62.7 mm to (6.98, 8.32)
- moved R214 62.7 mm to (11.7, 8.32)
- moved R233 61.9 mm to (21.2, 8.72)
- moved R245 61.9 mm to (16.5, 8.72)
- moved R223 58.8 mm to (26.0, 10.3)
- moved C210 57.0 mm to (6.98, 11.3)
- moved C213 57.0 mm to (11.7, 11.3)
- moved R215 56.2 mm to (16.5, 11.7)
- moved R239 56.2 mm to (21.2, 11.7)
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- renumbered R201 to R209, R202 to R210, R203 to R211, R204 to R212, R205 to R213, RV201 to RV203, RV203 to RV204, RV202 to RV205, RV204 to RV206
Connections:
- C214 pad 2: Net-(C210-Pad2) (its old number) -> /KicadJE_AteOhAte2/Coupling
- Q202 pad 2: Net-(Q201-Pad2) -> /KicadJE_AteOhAte2/PNP_E
- Q204 pad 1: Net-(Q203-Pad1) (its old number) -> Net-(Q204-Pad1)
- Q205 pad 1: (no net) -> /KicadJE_AteOhAte2/PNP_B
- Q205 pad 2: (no net) -> /KicadJE_AteOhAte2/PNP_E
- Q205 pad 3: (no net) -> /KicadJE_AteOhAte2/Coupling
- R228 pad 2: Net-(Q201-Pad2) -> /KicadJE_AteOhAte2/PNP_E
- R229 pad 1: Net-(Q204-PadB) -> /KicadJE_AteOhAte2/PNP_B
- R229 pad 2: Net-(Q201-Pad2) -> /KicadJE_AteOhAte2/PNP_E
- R236 pad 2: Net-(Q204-PadB) -> /KicadJE_AteOhAte2/PNP_B
- R237 pad 1: GND -> Net-(Q204-Pad1)
- R237 pad 2: Net-(Q203-Pad1) (its old number) -> GND
- R238 pad 2: Net-(C210-Pad2) (its old number) -> /KicadJE_AteOhAte2/Coupling
- R239 pad 2: Net-(C210-Pad2) (its old number) -> /KicadJE_AteOhAte2/Coupling
- R240 pad 2: Net-(Q203-Pad1) (its old number) -> Net-(Q204-Pad1)

Commit message: Test points for adj
Parts:
- moved JP201 138.7 mm to (81.0, 74.0), turned to 90 degrees
- moved RV202 135.3 mm to (85.0, 69.0)
- moved RV201 129.7 mm to (85.0, 53.0)
- moved R244 121.0 mm to (85.0, 81.0)
- moved R204 118.5 mm to (79.0, 60.0), turned to 180 degrees
- moved R243 115.2 mm to (80.0, 81.0)
- moved Q201 113.6 mm to (71.0, 54.0), turned to 90 degrees
- moved R202 108.1 mm to (75.0, 54.0)
- moved C208 106.6 mm to (70.0, 77.0), turned to 180 degrees
- moved C216 106.6 mm to (80.0, 86.0), turned to 180 degrees
- moved R201 106.2 mm to (75.0, 64.0)
- moved R205 102.9 mm to (75.0, 68.0)
- moved R203 102.3 mm to (79.0, 64.0)
- moved R206 102.0 mm to (71.0, 60.0)
- moved R207 100.7 mm to (75.0, 77.0), turned to 180 degrees
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Other:
- outline, holes or cut-outs redrawn
- board text added: "Reg noise to 130mV"
