File: KicadJE_AteOhAte/_autosave-KicadJE_AteOhAte.kicad_pcb (KiCad board)
At the start: 2 copper layers, 100 x 100 mm, 197 parts, among them J201 In_Accent, J202 In Gate, J203 Out Tom, J301 PJRAS2X2S01AUX, P201 Doepfer_Power_10pin, Q201 MMBT2222A, Q202 MMBT2222A, Q203 MMBT2222A, Q204 MMBT2222A, Q205 MMBT2907A, Q206 MMBT2222A, Q207 MMBT2222A, SW201 Con/Tom, U201 TL072, U202 TL072, U203 TL072, U301 TL072, U302 TL072, U303 TL072

Commit message: Fused RIAA SCH
Parts:
- removed D303: LED, LED_THT:LED_D3.0mm
- added C345: 470u, Capacitor_THT:CP_Radial_D13.0mm_P5.00mm, F.Cu at (116.0, 65.5)
- added C346: 470u, Capacitor_THT:CP_Radial_D13.0mm_P5.00mm, F.Cu at (116.0, 79.0)
- added J302: Conn_01x03, TerminalBlock:TerminalBlock_bornier-3_P5.08mm, F.Cu at (105.0, 79.5)
- added R329: 1R1, Resistor_SMD:R_0805_2012Metric_Pad1.15x1.40mm_HandSolder, B.Cu at (116.0, 62.0)
- added R330: 1R1, Resistor_SMD:R_0805_2012Metric_Pad1.15x1.40mm_HandSolder, B.Cu at (116.0, 87.5)
- C302, C316: footprint Capacitor_THT:CP_Radial_D6.3mm_P2.50mm -> Capacitor_SMD:CP_Elec_8x6.5
- C303, C306, C307, C308, C310, C311, C312, C313, C318, C319, C322, C323, C324, C326, C327, C328, C333, C334, C335, C336, C337, C338, C339, C340, C341, C342, D301, D302, H302, H304, R301, R302, R303, R304, R305, R306, R307, R308, R309, R310, R311, R312, R313, R314, R315, R316, R317, R318, R319, R320, R321, R322, R323, R324, R325, R326, R327, R328, U301, U302, U303: moved to B.Cu
- C331, C343: footprint Capacitor_THT:CP_Radial_D6.3mm_P2.50mm -> Capacitor_THT:CP_Radial_D8.0mm_P3.50mm
- C332, C344: value 10u -> 22u; footprint Capacitor_THT:CP_Radial_D6.3mm_P2.50mm -> Capacitor_THT:CP_Radial_D8.0mm_P3.50mm
- moved C310 161.5 mm to (221.9, 149.3)
- moved C339 161.5 mm to (226.7, 149.3)
- moved U301 156.9 mm to (188.7, 146.9)
- moved U302 156.9 mm to (178.0, 146.9)
- moved C338 155.8 mm to (221.9, 146.3)
- moved R301 155.8 mm to (226.7, 146.3)
- moved C333 150.2 mm to (221.9, 143.4)
- moved R305 150.2 mm to (226.7, 143.4)
- moved C306 146.5 mm to (215.2, 141.4)
- moved R310 144.6 mm to (220.0, 140.4)
- moved R322 144.6 mm to (224.7, 140.4)
- moved H304 143.6 mm to (209.9, 139.9)
- moved C340 140.8 mm to (215.2, 138.5)
- moved R320 138.9 mm to (226.6, 137.5)
- moved R324 138.9 mm to (221.9, 137.5)
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Connections:
- D304 pad 1: (no net) -> /KicadJE_AteOhAte3/-PSU
- R327 pad 2: (no net) -> /KicadJE_AteOhAte3/+PSU
