File: KicadJE_AteOhAte/KicadJE_AteOhAte.kicad_pcb (KiCad board)
At the start: 2 copper layers, 100 x 100 mm, 106 parts, among them J201 In_Accent, J202 In Gate, J203 Out Tom, P201 Doepfer_Power_10pin, Q201 MMBT2222A, Q202 MMBT2222A, Q203 MMBT2222A, Q204 MMBT2222A, Q205 MMBT2907A, Q206 MMBT2222A, Q207 MMBT2222A, SW201 Con/Tom, U201 TL072, U202 TL072, U203 TL072

Commit message: PCB before copper fill
Parts:
- added C301: 10n, Capacitor_SMD:C_0805_2012Metric_Pad1.15x1.40mm_HandSolder, F.Cu at (186.5, -0.57)
- added C302: 10n, Capacitor_SMD:C_0805_2012Metric_Pad1.15x1.40mm_HandSolder, F.Cu at (157.4, 25.9)
- added C303: 10n, Capacitor_SMD:C_0805_2012Metric_Pad1.15x1.40mm_HandSolder, F.Cu at (182.3, 2.38)
- added C304: 10n, Capacitor_SMD:C_0805_2012Metric_Pad1.15x1.40mm_HandSolder, F.Cu at (163.1, 20.0)
- added C305: 1u, Capacitor_SMD:C_0805_2012Metric_Pad1.15x1.40mm_HandSolder, F.Cu at (177.1, 6.23)
- added C306: 1u, Capacitor_SMD:C_0805_2012Metric_Pad1.15x1.40mm_HandSolder, F.Cu at (186.5, -3.52)
- added C307: 1u, Capacitor_SMD:C_0805_2012Metric_Pad1.15x1.40mm_HandSolder, F.Cu at (170.6, 11.8)
- added C308: 100n, Capacitor_SMD:C_0805_2012Metric_Pad1.15x1.40mm_HandSolder, F.Cu at (151.5, 30.7)
- added C309: 100n, Capacitor_SMD:C_0805_2012Metric_Pad1.15x1.40mm_HandSolder, F.Cu at (158.3, 20.0)
- added C310: 1u, Capacitor_SMD:C_0805_2012Metric_Pad1.15x1.40mm_HandSolder, F.Cu at (164.3, 16.7)
- added C311: 100n, Capacitor_SMD:C_0805_2012Metric_Pad1.15x1.40mm_HandSolder, F.Cu at (158.3, 22.9)
- added C312: 100n, Capacitor_SMD:C_0805_2012Metric_Pad1.15x1.40mm_HandSolder, F.Cu at (181.7, -0.57)
- added C313: 1u, Capacitor_SMD:C_0805_2012Metric_Pad1.15x1.40mm_HandSolder, F.Cu at (177.6, 2.98)
- added C314: 1u, Capacitor_SMD:C_0805_2012Metric_Pad1.15x1.40mm_HandSolder, F.Cu at (181.7, -3.52)
- added D301: LL4148, Diode_SMD:D_MiniMELF, F.Cu at (165.7, 4.38)
- added D302: LL4148, Diode_SMD:D_MiniMELF, F.Cu at (159.1, 10.9)
- added D303: LED, LED_THT:LED_D3.0mm, F.Cu at (170.5, 7.53)
- added D304: LL4148, Diode_SMD:D_MiniMELF, F.Cu at (169.8, -3.37)
- added D305: LL4148, Diode_SMD:D_MiniMELF, F.Cu at (172.0, 3.13)
- added D306: LL4148, Diode_SMD:D_MiniMELF, F.Cu at (176.2, -0.12)
- added D307: LL4148, Diode_SMD:D_MiniMELF, F.Cu at (145.9, 28.6)
- added D308: LL4148, Diode_SMD:D_MiniMELF, F.Cu at (176.2, -3.37)
- added D309: LL4148, Diode_SMD:D_MiniMELF, F.Cu at (165.7, 7.63)
- added D310: LED, LED_THT:LED_D3.0mm, F.Cu at (150.8, 26.5)
- added D311: D_Zener, Diode_SMD:D_MiniMELF, F.Cu at (145.9, 25.3)
- added D312: D_Zener, Diode_SMD:D_MiniMELF, F.Cu at (169.8, -0.12)
- added H201: 2,5mm, MountingHole:MountingHole_2.5mm_Pad_Via, F.Cu at (128.8, 38.9)
- added H202: 2,5mm, MountingHole:MountingHole_2.5mm_Pad_Via, F.Cu at (135.3, 38.9)
- added H203: 2,2mm, MountingHole:MountingHole_2.2mm_M2_Pad_Via, F.Cu at (128.5, 45.2)
- added H204: 2,2mm, MountingHole:MountingHole_2.2mm_M2_Pad_Via, F.Cu at (134.4, 45.2)
- added H301: 2,5mm, MountingHole:MountingHole_2.5mm_Pad_Via, F.Cu at (159.2, 6.03)
- added H302: 2,2mm, MountingHole:MountingHole_2.2mm_M2_Pad_Via, F.Cu at (158.9, 15.5)
- added H303: 2,5mm, MountingHole:MountingHole_2.5mm_Pad_Via, F.Cu at (139.5, 27.0)
- added H304: 2,2mm, MountingHole:MountingHole_2.2mm_M2_Pad_Via, F.Cu at (165.3, 12.3)
- added J301: Out 1, AJ-Dropbox-Kicad:PJ301SM, F.Cu at (150.9, 15.9)
- added J302: In_1, AJ-Dropbox-Kicad:PJ301SM, F.Cu at (150.9, 1.58)
- added J303: Out 2, AJ-Dropbox-Kicad:PJ301SM, F.Cu at (130.6, 1.58)
- added J304: In 2, AJ-Dropbox-Kicad:PJ301SM, F.Cu at (130.6, 15.9)
- added J305: Out 1 Final, AJ-Dropbox-Kicad:PJ301SM, F.Cu at (140.7, 1.58)
- added J306: Out 2 Final, AJ-Dropbox-Kicad:PJ301SM, F.Cu at (140.7, 15.9)
- added R301: 1k, Resistor_SMD:R_0805_2012Metric_Pad1.15x1.40mm_HandSolder, F.Cu at (187.1, 5.33)
- added R302: 10k, Resistor_SMD:R_0805_2012Metric_Pad1.15x1.40mm_HandSolder, F.Cu at (161.0, 28.8)
- added R303: 10k, Resistor_SMD:R_0805_2012Metric_Pad1.15x1.40mm_HandSolder, F.Cu at (181.9, 8.28)
- added R304: 1k, Resistor_SMD:R_0805_2012Metric_Pad1.15x1.40mm_HandSolder, F.Cu at (167.8, 22.6)
- added R305: 1k, Resistor_SMD:R_0805_2012Metric_Pad1.15x1.40mm_HandSolder, F.Cu at (175.4, 15.1)
- added R306: 1k, Resistor_SMD:R_0805_2012Metric_Pad1.15x1.40mm_HandSolder, F.Cu at (175.4, 12.1)
- added R307: 10k, Resistor_SMD:R_0805_2012Metric_Pad1.15x1.40mm_HandSolder, F.Cu at (187.1, 2.38)
- added R308: 10k, Resistor_SMD:R_0805_2012Metric_Pad1.15x1.40mm_HandSolder, F.Cu at (172.6, 18.0)
- added R309: 10R, Resistor_SMD:R_0805_2012Metric_Pad1.15x1.40mm_HandSolder, F.Cu at (162.1, 25.9)
- added R310: 1k, Resistor_SMD:R_0805_2012Metric_Pad1.15x1.40mm_HandSolder, F.Cu at (182.3, 5.33)
- added R311: 1k, Resistor_SMD:R_0805_2012Metric_Pad1.15x1.40mm_HandSolder, F.Cu at (177.1, 9.18)
- added R312: 10k, Resistor_SMD:R_0805_2012Metric_Pad1.15x1.40mm_HandSolder, F.Cu at (156.2, 30.7)
- added R313: 100k, Resistor_SMD:R_0805_2012Metric_Pad1.15x1.40mm_HandSolder, F.Cu at (163.1, 22.9)
- added R314: 10k, Resistor_SMD:R_0805_2012Metric_Pad1.15x1.40mm_HandSolder, F.Cu at (177.3, 18.0)
- added R315: 100k, Resistor_SMD:R_0805_2012Metric_Pad1.15x1.40mm_HandSolder, F.Cu at (167.8, 19.7)
- added R316: 1k, Resistor_SMD:R_0805_2012Metric_Pad1.15x1.40mm_HandSolder, F.Cu at (182.1, 18.0)
- added R317: 10k, Resistor_SMD:R_0805_2012Metric_Pad1.15x1.40mm_HandSolder, F.Cu at (189.6, 11.2)
- added R318: 10k, Resistor_SMD:R_0805_2012Metric_Pad1.15x1.40mm_HandSolder, F.Cu at (177.3, 23.9)
- added R319: 1k, Resistor_SMD:R_0805_2012Metric_Pad1.15x1.40mm_HandSolder, F.Cu at (171.6, 26.9)
- added R320: Open, Resistor_SMD:R_0805_2012Metric_Pad1.15x1.40mm_HandSolder, F.Cu at (184.9, 14.2)
- added R321: Open, Resistor_SMD:R_0805_2012Metric_Pad1.15x1.40mm_HandSolder, F.Cu at (177.3, 21.0)
- added R322: 1k, Resistor_SMD:R_0805_2012Metric_Pad1.15x1.40mm_HandSolder, F.Cu at (184.9, 11.2)
- added R323: 10R, Resistor_SMD:R_0805_2012Metric_Pad1.15x1.40mm_HandSolder, F.Cu at (180.1, 12.1)
- added R324: 1k, Resistor_SMD:R_0805_2012Metric_Pad1.15x1.40mm_HandSolder, F.Cu at (172.6, 23.9)
- added R325: 0R, Resistor_SMD:R_0805_2012Metric_Pad1.15x1.40mm_HandSolder, F.Cu at (186.6, 8.28)
- added R326: 0R, Resistor_SMD:R_0805_2012Metric_Pad1.15x1.40mm_HandSolder, F.Cu at (165.7, 28.8)
- added R327: 10k, Resistor_SMD:R_0805_2012Metric_Pad1.15x1.40mm_HandSolder, F.Cu at (180.1, 15.1)
- added R328: OPEN, Resistor_SMD:R_0805_2012Metric_Pad1.15x1.40mm_HandSolder, F.Cu at (172.6, 21.0)
- added R329: 10k, Resistor_SMD:R_0805_2012Metric_Pad1.15x1.40mm_HandSolder, F.Cu at (166.9, 25.9)
- added R330: OPEN, Resistor_SMD:R_0805_2012Metric_Pad1.15x1.40mm_HandSolder, F.Cu at (170.6, 14.7)
- added TP203: Coupling, TestPoint:TestPoint_Pad_1.5x1.5mm, F.Cu at (94.0, 103.0)
- added U301: TL072, AJ-Dropbox-Kicad:AJ_SO-8_5.3x6.2mm_P1.27mm, F.Cu at (130.9, 27.6)
- added U302: TL072, AJ-Dropbox-Kicad:AJ_SO-8_5.3x6.2mm_P1.27mm, F.Cu at (161.3, -1.12)
- moved D208 76.9 mm to (92.5, 102.0), turned to 270 degrees
- moved C215 74.6 mm to (96.0, 86.5)
- moved C218 74.6 mm to (91.5, 81.0)
- moved Q207 74.6 mm to (91.0, 86.5)
- moved R242 74.6 mm to (96.0, 89.5)
- moved R245 74.6 mm to (96.0, 81.0)
- moved R250 74.6 mm to (96.0, 83.5)
- moved C219 73.9 mm to (83.5, 93.0), turned to 180 degrees
- moved R248 73.4 mm to (83.5, 89.5), turned to 180 degrees
- moved R249 73.2 mm to (83.5, 86.0), turned to 0 degrees
- moved R244 1.53 mm to (83.5, 81.0)
- moved C212 0.75 mm to (57.0, 109.8)
- moved C216 0.50 mm to (79.5, 86.0)
- moved R243 0.50 mm to (79.5, 81.0)
Routing:
- net Net-(C210-Pad2): track 39.8 -> 99.5 mm, vias 0 -> 2
- net Net-(C218-Pad1): track 0.00 -> 54.1 mm, vias 0 -> 4
- net Net-(C209-Pad2): track 9.72 -> 56.0 mm, vias 0 -> 2
- net +12V: track 197.0 -> 237.6 mm
- net /KicadJE_AteOhAte2/Coupling: track 5.01 -> 41.4 mm, vias 0 -> 5
- net Net-(C212-Pad1): track 13.9 -> 48.4 mm, vias 0 -> 5
- net Net-(C212-Pad2): track 23.7 -> 52.9 mm, vias 0 -> 4
- net GND: track 95.0 -> 121.9 mm, vias 0 -> 1
- net Net-(C210-Pad1): track 3.66 -> 25.3 mm, vias 0 -> 4
- net Net-(R230-Pad2): track 0.00 -> 20.8 mm
- net Net-(C219-Pad1): track 0.00 -> 14.9 mm
- net Net-(D208-Pad2): track 0.00 -> 13.8 mm
- net Net-(C209-Pad1): track 0.00 -> 10.7 mm
- net Net-(C216-Pad2): track 0.00 -> 8.27 mm
- net NoiseIn: track 0.00 -> 7.41 mm
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
Commit message: RIAA SCH started
Parts:
- removed H203: 2,2mm, MountingHole:MountingHole_2.2mm_M2_Pad_Via
- added G***: LOGO, AJ:Johansen_engineering_logo_25mm_front_neg5, B.Cu at (94.5, 138.0)
- added G***: LOGO, AJ:Johansen_engineering_logo_25mm_front_neg5, F.Cu at (94.2, 138.5)
- D204: value D_Zener -> Zener
- moved H202 106.9 mm to (104.2, 141.2)
- moved H201 103.2 mm to (140.0, 141.5)
- moved H204 98.8 mm to (88.8, 132.8)
- moved H301 55.9 mm to (140.0, 58.5)
- moved H303 47.3 mm to (104.2, 58.5)
Routing:
- net GND: track 121.9 -> 198.5 mm, vias 1 -> 77
- net Net-(C205-Pad2): track 0.00 -> 13.7 mm
- net (no net): track 0.00 -> 4.81 mm, vias 0 -> 3
- net +12V: track 237.6 -> 238.2 mm
- added copper zone on B.Cu, net GND
- added copper zone on F.Cu, net GND
Other:
- outline, holes or cut-outs redrawn
- board text added: "DRUM_Ate0Ate_Tom_1 Rev A - 25/09-2019 Johansen Engineering"
