File: KicadJE_AteOhAte/KicadJE_AteOhAte.kicad_pcb (KiCad board)
At the start: 2 copper layers, 100 x 100 mm, 203 parts, among them J201 In_Accent, J202 In Gate, J203 Out Tom, J301 PJRAS2X2S01AUX, J302 Conn_01x03, P201 Doepfer_Power_10pin, Q201 MMBT2222A, Q202 MMBT2222A, Q203 MMBT2222A, Q204 MMBT2222A, Q205 MMBT2907A, Q206 MMBT2222A, Q207 MMBT2222A, SW201 Con/Tom, U201 TL072, U202 TL072, U203 TL072, U301 TL072, U302 TL072, U303 TL072

Commit message: Ate0Ate Tom Labels
Parts:
- D204: value D_Zener -> Zener

Commit message: Label tweaks
Parts:
- D203: value D_Zener -> Zener
Changed lines of the file:
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@@
     )
     (fp_text value 47n (at 3.5 0 180) (layer B.SilkS)
-      (effects (font (size 1 1) (thickness 0.15)) (justify mirror))
+      (effects (font (size 0.9 0.9) (thickness 0.15)) (justify mirror))
     )
     (fp_text user %R (at 0 0 180) (layer B.Fab)
@@
     (tags SOT-23)
     (attr smd)
-    (fp_text reference Q204 (at 0 2.3 270) (layer B.SilkS)
+    (fp_text reference Q204 (at 0.8 3.8) (layer B.SilkS)
       (effects (font (size 1 1) (thickness 0.15)) (justify mirror))
     )
@@
     (tags "capacitor handsolder")
     (attr smd)
-    (fp_text reference C202 (at 0 1.65 270) (layer B.SilkS)
-      (effects (font (size 1 1) (thickness 0.15)) (justify mirror))
+    (fp_text reference C202 (at -2.3 -0.05) (layer B.SilkS)
+      (effects (font (size 0.9 0.9) (thickness 0.15)) (justify mirror))
     )
-    (fp_text value 100n (at 0 -1.65 270) (layer B.Fab)
-      (effects (font (size 1 1) (thickness 0.15)) (justify mirror))
+    (fp_text value 100n (at 2.5 -0.05) (layer B.SilkS)
+      (effects (font (size 0.8 0.8) (thickness 0.15)) (justify mirror))
     )
     (fp_text user %R (at 0 0 270) (layer B.Fab)
@@
       (effects (font (size 1 1) (thickness 0.15)) (justify mirror))
     )
-    (fp_text value D_Zener (at 0.95 -3.25) (layer B.Fab)
-      (effects (font (size 1 1) (thickness 0.15)) (justify mirror))
+    (fp_text value Zener (at 0.4 -2.8) (layer B.SilkS)
+      (effects (font (size 0.7 0.7) (thickness 0.15)) (justify mirror))
     )
     (fp_line (start -2.65 -1.1) (end -2.65 1.1) (layer B.CrtYd) (width 0.05))
@@
     (tags "resistor handsolder")
     (attr smd)
-    (fp_text reference R209 (at 0 1.65) (layer B.SilkS)
+    (fp_text reference R209 (at -0.15 1.65) (layer B.SilkS)
       (effects (font (size 1 1) (thickness 0.15)) (justify mirror))
     )
@@
     (tags "resistor handsolder")
     (attr smd)
-    (fp_text reference R210 (at 0 1.65) (layer B.SilkS)
+    (fp_text reference R210 (at 0.1 1.65) (layer B.SilkS)
       (effects (font (size 1 1) (thickness 0.15)) (justify mirror))
     )
-    (fp_text value OPEN (at 0 2.825001) (layer B.SilkS)
-      (effects (font (size 1 1) (thickness 0.15)) (justify mirror))
+    (fp_text value OPEN (at 0 3.125001) (layer B.SilkS)
+      (effects (font (size 0.8 0.8) (thickness 0.15)) (justify mirror))
     )
     (fp_line (start -1 -0.6) (end -1 0.6) (layer B.Fab) (width 0.1))
@@
     (tags "capacitor handsolder")
     (attr smd)
-    (fp_text reference C217 (at -3.75 1) (layer B.SilkS)
+    (fp_text reference C217 (at -3.7 0) (layer B.SilkS)
       (effects (font (size 1 1) (thickness 0.15)) (justify mirror))
     )
     (fp_text value 10n (at 1.25 1.5) (layer B.SilkS)
-      (effects (font (size 1 1) (thickness 0.15)) (justify mirror))
+      (effects (font (size 0.8 0.8) (thickness 0.15)) (justify mirror))
     )
     (fp_line (start -1 -0.6) (end -1 0.6) (layer B.Fab) (width 0.1))
@@
     (tags SOT-23)
     (attr smd)
-    (fp_text reference Q203 (at 0 2.5 90) (layer B.SilkS)
+    (fp_text reference Q203 (at 1.6 2.6 180) (layer B.SilkS)
       (effects (font (size 1 1) (thickness 0.15)) (justify mirror))
     )
@@
     (tags SOT-23)
     (attr smd)
-    (fp_text reference Q206 (at 0 2.5 90) (layer B.SilkS)
+    (fp_text reference Q206 (at 1.8 2.7 180) (layer B.SilkS)
       (effects (font (size 1 1) (thickness 0.15)) (justify mirror))
     )
@@
     )
     (fp_text value 100k (at -0.9 2.75 180) (layer B.SilkS)
-      (effects (font (size 1 1) (thickness 0.15)) (justify mirror))
+      (effects (font (size 0.8 0.8) (thickness 0.15)) (justify mirror))
     )
     (fp_line (start -1 -0.6) (end -1 0.6) (layer B.Fab) (width 0.1))
@@
     )
     (fp_text value 4k7 (at -2.5 1.25 180) (layer B.SilkS)
-      (effects (font (size 1 1) (thickness 0.15)) (justify mirror))
+      (effects (font (size 0.8 0.8) (thickness 0.15)) (justify mirror))
     )
     (fp_line (start -1 -0.6) (end -1 0.6) (layer B.Fab) (width 0.1))
@@
     (tags "resistor handsolder")
     (attr smd)
-    (fp_text reference R237 (at 0 1.65) (layer B.SilkS)
+    (fp_text reference R237 (at -0.275 -1.5) (layer B.SilkS)
       (effects (font (size 1 1) (thickness 0.15)) (justify mirror))
     )
-    (fp_text value 10k (at 0 -1.65) (layer B.SilkS)
+    (fp_text value 10k (at -0.175 1.7) (layer B.SilkS)
       (effects (font (size 1 1) (thickness 0.15)) (justify mirror))
     )
@@
       (effects (font (size 1 1) (thickness 0.15)) (justify mirror))
     )
-    (fp_text value 22k (at 0 -1.65 90) (layer B.Fab)
-      (effects (font (size 1 1) (thickness 0.15)) (justify mirror))
+    (fp_text value 22k (at -2.525 0.2 180) (layer B.SilkS)
+      (effects (font (size 0.8 0.8) (thickness 0.15)) (justify mirror))
     )
     (fp_text user %R (at 0 0 90) (layer B.Fab)
@@
       (effects (font (size 1 1) (thickness 0.15)) (justify mirror))
     )
-    (fp_text value 10k (at 0 -1.65 180) (layer B.Fab)
-      (effects (font (size 1 1) (thickness 0.15)) (justify mirror))
+    (fp_text value 10k (at 0 -1.65 180) (layer B.SilkS)
+      (effects (font (size 0.8 0.8) (thickness 0.15)) (justify mirror))
     )
     (fp_line (start -1 -0.6) (end -1 0.6) (layer B.Fab) (width 0.1))
@@
     (tags "resistor handsolder")
     (attr smd)
-    (fp_text reference R241 (at 0 1.65 270) (layer B.SilkS)
-      (effects (font (size 1 1) (thickness 0.15)) (justify mirror))
+    (fp_text reference R241 (at -2.3 0.1) (layer B.SilkS)
+      (effects (font (size 0.9 0.9) (thickness 0.15)) (justify mirror))
     )
-    (fp_text value 22k (at 3.25 0 270) (layer B.SilkS)
-      (effects (font (size 1 1) (thickness 0.15)) (justify mirror))
+    (fp_text value 22k (at 2.5 0) (layer B.SilkS)
+      (effects (font (size 0.8 0.8) (thickness 0.15)) (justify mirror))
     )
     (fp_line (start -1 -0.6) (end -1 0.6) (layer B.Fab) (width 0.1))
@@
     )
     (fp_text value 100k (at -1 -1.5 180) (layer B.SilkS)
-      (effects (font (size 1 1) (thickness 0.15)) (justify mirror))
+      (effects (font (size 0.8 0.8) (thickness 0.15)) (justify mirror))
     )
     (fp_text user %R (at 0 0 180) (layer B.Fab)
@@
       (effects (font (size 1 1) (thickness 0.15)) (justify mirror))
     )
-    (fp_text value 10k (at 2.5 0 90) (layer B.SilkS)
-      (effects (font (size 1 1) (thickness 0.15)) (justify mirror))
+    (fp_text value 10k (at 3 0.05 180) (layer B.SilkS)
+      (effects (font (size 0.8 0.8) (thickness 0.15)) (justify mirror))
     )
     (fp_line (start -1 -0.6) (end -1 0.6) (layer B.Fab) (width 0.1))
@@
     )
     (fp_text value C6 (at 2.875 1.124999 180) (layer B.SilkS)
-      (effects (font (size 1 1) (thickness 0.15)) (justify mirror))
+      (effects (font (size 0.8 0.8) (thickness 0.15)) (justify mirror))
     )
     (fp_line (start -1 -0.6) (end -1 0.6) (layer B.Fab) (width 0.1))
@@
     )
     (fp_text value C7 (at 0 3 180) (layer B.SilkS)
-      (effects (font (size 1 1) (thickness 0.15)) (justify mirror))
+      (effects (font (size 0.9 0.9) (thickness 0.15)) (justify mirror))
     )
     (fp_line (start -1 -0.6) (end -1 0.6) (layer B.Fab) (width 0.1))
@@
     )
     (fp_text value 4k7 (at 0.2 1.5) (layer B.SilkS)
-      (effects (font (size 1 1) (thickness 0.15)) (justify mirror))
+      (effects (font (size 0.8 0.8) (thickness 0.15)) (justify mirror))
     )
     (fp_text user %R (at 0 0) (layer B.Fab)
@@
     )
     (fp_text value 22k (at 0.275 3 180) (layer B.SilkS)
-      (effects (font (size 1 1) (thickness 0.15)) (justify mirror))
+      (effects (font (size 0.9 0.9) (thickness 0.15)) (justify mirror))
     )
     (fp_text user %R (at 0 0 180) (layer B.Fab)
@@
       (effects (font (size 1 1) (thickness 0.15)) (justify mirror))
     )
-    (fp_text value MMBT2907A (at 0 -2.5 270) (layer B.SilkS)
+    (fp_text value MMBT2907A (at 0.05 -2.8 270) (layer B.SilkS)
       (effects (font (size 1 1) (thickness 0.15)) (justify mirror))
     )
@@
     (effects (font (size 2.5 2.5) (thickness 0.625)))
   )
-  (gr_text "DRUM_Ate0Ate_Tom_1\nRev A - 25/09-2019\nJohansen Engineering" (at 69.75 111.25 90) (layer B.SilkS)
-    (effects (font (size 1.3 1.25) (thickness 0.3)) (justify mirror))
+  (gr_text "DRUM_Ate0Ate_Tom_1\nRev A - 25/09-2019\nJohansen Engineering" (at 71.1 110.5 90) (layer B.SilkS)
+    (effects (font (size 1.3 1.2) (thickness 0.3)) (justify mirror))
   )
   (gr_line (start 100 69.5) (end 150 69.5) (layer Dwgs.User) (width 0.15))

Commit message: Label tweaks
Parts:
- removed H203, H302, H304: 2,2mm, MountingHole:MountingHole_2.2mm_M2_Pad_Via
- added C220: 10u, Capacitor_SMD:C_1206_3216Metric_Pad1.42x1.75mm_HandSolder, B.Cu at (89.1, 64.8)
- added C221: 10u, Capacitor_SMD:C_1206_3216Metric_Pad1.42x1.75mm_HandSolder, B.Cu at (89.1, 58.6)
- D203, D204: value Zener -> D_Zener
Routing:
- net GND: track 216.2 -> 225.6 mm, vias 144 -> 145
- net -12V: track 223.1 -> 225.6 mm
