File: KicadJE_AteOhAte/KicadJE_AteOhAte3.sch (KiCad schematic (older format))
At the start: 68 parts, among them J303 Out 1, J304 In_1, J305 Out 2, J306 In 2, J307 Out 1 Final, J308 Out 2 Final, U301 TL072, U302 TL072

Commit message: 2nd stage Tom sch initiated
Parts:
- renumbered J303 to J301, J304 to J302, J305 to J303, J306 to J304, J307 to J305, J308 to J306
Changed lines of the file:
@@
 AR Path="/5CF11B19/5D513A01" Ref="#PWR?"  Part="1"
 AR Path="/5D4DB58B/5D513A01" Ref="#PWR?"  Part="1"
-AR Path="/5D4DB615/5D513A01" Ref="#PWR0317"  Part="1"
-F 0 "#PWR0317" H 1650 6625 50  0001 C CNN
+AR Path="/5D4DB615/5D513A01" Ref="#PWR0311"  Part="1"
+F 0 "#PWR0311" H 1650 6625 50  0001 C CNN
 F 1 "GND" H 1655 6702 50  0000 C CNN
 F 2 "" H 1650 6875 50  0001 C CNN
@@
 	1650 6875 2525 6875
 $Comp
-L power:+12V #PWR0316
+L power:+12V #PWR0310
 U 1 1 5D58F7D5
 P 2725 6575
-F 0 "#PWR0316" H 2725 6425 50  0001 C CNN
+F 0 "#PWR0310" H 2725 6425 50  0001 C CNN
 F 1 "+12V" H 2740 6748 50  0000 C CNN
 F 2 "" H 2725 6575 50  0001 C CNN
@@
 $EndComp
 $Comp
-L power:-12V #PWR0318
+L power:-12V #PWR0312
 U 1 1 5D59049F
 P 2725 7175
-F 0 "#PWR0318" H 2725 7275 50  0001 C CNN
+F 0 "#PWR0312" H 2725 7275 50  0001 C CNN
 F 1 "-12V" H 2740 7348 50  0000 C CNN
 F 2 "" H 2725 7175 50  0001 C CNN
@@
 P 6250 6225
 AR Path="/5CF11B19/5D7994F9" Ref="J?"  Part="1"
-AR Path="/5D4DB615/5D7994F9" Ref="J303"  Part="1"
-F 0 "J303" H 6017 6296 50  0000 R CNN
+AR Path="/5D4DB615/5D7994F9" Ref="J301"  Part="1"
+F 0 "J301" H 6017 6296 50  0000 R CNN
 F 1 "Out 1" H 6017 6205 50  0000 R CNN
 F 2 "AJ-Dropbox-Kicad:PJ301SM" H 6250 6225 50  0001 C CNN
@@
 P 6250 6625
 AR Path="/5CF11B19/5D7994FF" Ref="J?"  Part="1"
-AR Path="/5D4DB615/5D7994FF" Ref="J305"  Part="1"
-F 0 "J305" H 6017 6696 50  0000 R CNN
+AR Path="/5D4DB615/5D7994FF" Ref="J303"  Part="1"
+F 0 "J303" H 6017 6696 50  0000 R CNN
 F 1 "Out 2" H 6017 6605 50  0000 R CNN
 F 2 "AJ-Dropbox-Kicad:PJ301SM" H 6250 6625 50  0001 C CNN
@@
 P 4675 6550
 AR Path="/5CF11B19/5D799508" Ref="J?"  Part="1"
-AR Path="/5D4DB615/5D799508" Ref="J304"  Part="1"
-F 0 "J304" H 4442 6621 50  0000 R CNN
+AR Path="/5D4DB615/5D799508" Ref="J302"  Part="1"
+F 0 "J302" H 4442 6621 50  0000 R CNN
 F 1 "In_1" H 4442 6530 50  0000 R CNN
 F 2 "AJ-Dropbox-Kicad:PJ301SM" H 4675 6550 50  0001 C CNN
@@
 P 5900 7475
 AR Path="/5CF11B19/5D79953C" Ref="#PWR?"  Part="1"
-AR Path="/5D4DB615/5D79953C" Ref="#PWR0320"  Part="1"
-F 0 "#PWR0320" H 5900 7225 50  0001 C CNN
+AR Path="/5D4DB615/5D79953C" Ref="#PWR0314"  Part="1"
+F 0 "#PWR0314" H 5900 7225 50  0001 C CNN
 F 1 "GND" H 5905 7302 50  0000 C CNN
 F 2 "" H 5900 7475 50  0001 C CNN
@@
 P 4325 7350
 AR Path="/5CF11B19/5D799544" Ref="#PWR?"  Part="1"
-AR Path="/5D4DB615/5D799544" Ref="#PWR0319"  Part="1"
-F 0 "#PWR0319" H 4325 7100 50  0001 C CNN
+AR Path="/5D4DB615/5D799544" Ref="#PWR0313"  Part="1"
+F 0 "#PWR0313" H 4325 7100 50  0001 C CNN
 F 1 "GND" H 4330 7177 50  0000 C CNN
 F 2 "" H 4325 7350 50  0001 C CNN
@@
 P 4675 7000
 AR Path="/5CF11B19/5D79954C" Ref="J?"  Part="1"
-AR Path="/5D4DB615/5D79954C" Ref="J306"  Part="1"
-F 0 "J306" H 4442 7071 50  0000 R CNN
+AR Path="/5D4DB615/5D79954C" Ref="J304"  Part="1"
+F 0 "J304" H 4442 7071 50  0000 R CNN
 F 1 "In 2" H 4442 6980 50  0000 R CNN
 F 2 "AJ-Dropbox-Kicad:PJ301SM" H 4675 7000 50  0001 C CNN
@@
 P 6250 7375
 AR Path="/5CF11B19/5D79956C" Ref="J?"  Part="1"
-AR Path="/5D4DB615/5D79956C" Ref="J308"  Part="1"
-F 0 "J308" H 6017 7446 50  0000 R CNN
+AR Path="/5D4DB615/5D79956C" Ref="J306"  Part="1"
+F 0 "J306" H 6017 7446 50  0000 R CNN
 F 1 "Out 2 Final" H 6017 7355 50  0000 R CNN
 F 2 "AJ-Dropbox-Kicad:PJ301SM" H 6250 7375 50  0001 C CNN
@@
 P 6250 7025
 AR Path="/5CF11B19/5D84994A" Ref="J?"  Part="1"
-AR Path="/5D4DB615/5D84994A" Ref="J307"  Part="1"
-F 0 "J307" H 6017 7096 50  0000 R CNN
+AR Path="/5D4DB615/5D84994A" Ref="J305"  Part="1"
+F 0 "J305" H 6017 7096 50  0000 R CNN
 F 1 "Out 1 Final" H 6017 7005 50  0000 R CNN
 F 2 "AJ-Dropbox-Kicad:PJ301SM" H 6250 7025 50  0001 C CNN
@@
 AR Path="/5CF11B19/5D88CF5A" Ref="#PWR?"  Part="1"
 AR Path="/5D4DB58B/5D88CF5A" Ref="#PWR?"  Part="1"
-AR Path="/5D4DB615/5D88CF5A" Ref="#PWR0315"  Part="1"
-F 0 "#PWR0315" H 7475 5200 50  0001 C CNN
+AR Path="/5D4DB615/5D88CF5A" Ref="#PWR0309"  Part="1"
+F 0 "#PWR0309" H 7475 5200 50  0001 C CNN
 F 1 "GND" H 7480 5277 50  0000 C CNN
 F 2 "" H 7475 5450 50  0001 C CNN
@@
 Connection ~ 7475 4650
 $Comp
-L power:+12V #PWR0313
+L power:+12V #PWR0307
 U 1 1 5D8A8AB9
 P 7050 4650
-F 0 "#PWR0313" H 7050 4500 50  0001 C CNN
+F 0 "#PWR0307" H 7050 4500 50  0001 C CNN
 F 1 "+12V" H 7065 4823 50  0000 C CNN
 F 2 "" H 7050 4650 50  0001 C CNN
@@
 AR Path="/5CF11B19/5D8B385E" Ref="#PWR?"  Part="1"
 AR Path="/5D4DB58B/5D8B385E" Ref="#PWR?"  Part="1"
-AR Path="/5D4DB615/5D8B385E" Ref="#PWR0314"  Part="1"
-F 0 "#PWR0314" H 4375 4850 50  0001 C CNN
+AR Path="/5D4DB615/5D8B385E" Ref="#PWR0308"  Part="1"
+F 0 "#PWR0308" H 4375 4850 50  0001 C CNN
 F 1 "GND" H 4380 4927 50  0000 C CNN
 F 2 "" H 4375 5100 50  0001 C CNN
@@
 Connection ~ 4375 4650
 $Comp
-L power:+12V #PWR0312
+L power:+12V #PWR0306
 U 1 1 5D8B3881
 P 3950 4650
-F 0 "#PWR0312" H 3950 4500 50  0001 C CNN
+F 0 "#PWR0306" H 3950 4500 50  0001 C CNN
 F 1 "+12V" H 3965 4823 50  0000 C CNN
 F 2 "" H 3950 4650 50  0001 C CNN
@@
 AR Path="/5CF11B19/5DA41BB2" Ref="#PWR?"  Part="1"
 AR Path="/5D4DB58B/5DA41BB2" Ref="#PWR?"  Part="1"
-AR Path="/5D4DB615/5DA41BB2" Ref="#PWR0306"  Part="1"
-F 0 "#PWR0306" H 9550 2850 50  0001 C CNN
+AR Path="/5D4DB615/5DA41BB2" Ref="#PWR0303"  Part="1"
+F 0 "#PWR0303" H 9550 2850 50  0001 C CNN
 F 1 "GND" H 9555 2927 50  0000 C CNN
 F 2 "" H 9550 3100 50  0001 C CNN
@@
 AR Path="/5CF11B19/5DB3EFD6" Ref="#PWR?"  Part="1"
 AR Path="/5D4DB58B/5DB3EFD6" Ref="#PWR?"  Part="1"
-AR Path="/5D4DB615/5DB3EFD6" Ref="#PWR0307"  Part="1"
-F 0 "#PWR0307" H 6875 3700 50  0001 C CNN
+AR Path="/5D4DB615/5DB3EFD6" Ref="#PWR0304"  Part="1"
+F 0 "#PWR0304" H 6875 3700 50  0001 C CNN
 F 1 "GND" H 6880 3777 50  0000 C CNN
 F 2 "" H 6875 3950 50  0001 C CNN
@@
 AR Path="/5CF11B19/5DB55B3C" Ref="#PWR?"  Part="1"
 AR Path="/5D4DB58B/5DB55B3C" Ref="#PWR?"  Part="1"
-AR Path="/5D4DB615/5DB55B3C" Ref="#PWR0310"  Part="1"
-F 0 "#PWR0310" H 3400 3900 50  0001 C CNN
+AR Path="/5D4DB615/5DB55B3C" Ref="#PWR0305"  Part="1"
+F 0 "#PWR0305" H 3400 3900 50  0001 C CNN
 F 1 "GND" H 3405 3977 50  0000 C CNN
 F 2 "" H 3400 4150 50  0001 C CNN

Commit message: RIAA SCH started
Parts:
- removed D311, D312: D_Zener, Diode_SMD:D_MiniMELF, symbol Device:D_Zener
- removed J302: In_1, AJ-Dropbox-Kicad:PJ301SM, symbol Connector:AudioJack2_SwitchT
- removed J304: In 2, AJ-Dropbox-Kicad:PJ301SM, symbol Connector:AudioJack2_SwitchT
- added J?: Conn_Coaxial_x2, symbol Connector:Conn_Coaxial_x2
Connections:
- net GND: now also J?.3 (EXT)
- net at R327.1: now also J?.1 (IN1)
- net at R329.1: now also J?.2 (IN2)
- net In_1: no longer names the net of R307.2
- net In_1: no longer C306.2
- net In_2: no longer names the net of R317.2
- net In_2: no longer C310.2
- net POT1_C: no longer names the net of R301.2, R305.1
- net POT1_L: no longer names the net of C301.1, D301.2 (A), D302.1 (K), R302.1, U301.6 (-)
- net POT2_C: no longer names the net of R304.1
- net POT2_L: no longer names the net of R303.1, U301.2 (-)
- net POT3_C: no longer names the net of R312.1, R318.2, R322.1, U302.7
- net POT3_L: no longer names the net of R316.1
- net POT4_C: no longer names the net of R319.2, R324.2, U302.1
- net POT4_L: no longer names the net of R314.1
- new net In_L: C306.2
- new net In_R: C310.2
Changed lines of the file:
@@
 encoding utf-8
 Sheet 3 3
-Title ""
-Date ""
-Rev ""
-Comp ""
+Title "RIAA"
+Date "2019-09-25"
+Rev "Rev A"
+Comp "Johansen Engineering"
 Comment1 ""
 Comment2 ""
@@
 	-1   0    0    -1
 $EndComp
-$Comp
-L Connector:AudioJack2_SwitchT J?
-U 1 1 5D799508
-P 4675 6550
-AR Path="/5CF11B19/5D799508" Ref="J?"  Part="1"
-AR Path="/5D4DB615/5D799508" Ref="J302"  Part="1"
-F 0 "J302" H 4442 6621 50  0000 R CNN
-F 1 "In_1" H 4442 6530 50  0000 R CNN
-F 2 "AJ-Dropbox-Kicad:PJ301SM" H 4675 6550 50  0001 C CNN
-F 3 "~" H 4675 6550 50  0001 C CNN
-F 4 "VC input" H 4675 6550 50  0001 C CNN "Function"
-	1    4675 6550
-	-1   0    0    -1
-$EndComp
-Wire Wire Line
-	4475 6450 4325 6450
 Wire Wire Line
 	6050 6125 5900 6125
@@
 $EndComp
 Wire Wire Line
-	4225 6550 4375 6550
-Wire Wire Line
 	5900 6125 5900 6525
 Connection ~ 3875 6550
@@
 	3875 6550 3925 6550
 Wire Wire Line
-	4325 6450 4325 6700
-Wire Wire Line
 	3875 6700 3925 6700
 Wire Wire Line
 	3875 6550 3875 6700
-Wire Wire Line
-	4225 6700 4325 6700
-Connection ~ 4325 6700
-Wire Wire Line
-	4325 6700 4325 6900
-Wire Wire Line
-	4475 6900 4325 6900
 $Comp
 L Device:R R?
@@
 	0    -1   -1   0
 $EndComp
-Wire Wire Line
-	4225 7000 4425 7000
 Connection ~ 3875 7000
 Wire Wire Line
 	3875 7000 3925 7000
 Wire Wire Line
-	4325 6900 4325 7150
-Wire Wire Line
 	3875 7150 3925 7150
 Wire Wire Line
 	3875 7000 3875 7150
-Wire Wire Line
-	4225 7150 4325 7150
-Connection ~ 4325 6900
 $Comp
 L power:GND #PWR?
@@
 L power:GND #PWR?
 U 1 1 5D799544
-P 4325 7350
+P 4800 7250
 AR Path="/5CF11B19/5D799544" Ref="#PWR?"  Part="1"
 AR Path="/5D4DB615/5D799544" Ref="#PWR0313"  Part="1"
-F 0 "#PWR0313" H 4325 7100 50  0001 C CNN
-F 1 "GND" H 4330 7177 50  0000 C CNN
-F 2 "" H 4325 7350 50  0001 C CNN
-F 3 "" H 4325 7350 50  0001 C CNN
-	1    4325 7350
-	1    0    0    -1
-$EndComp
-Connection ~ 4325 7150
-$Comp
-L Connector:AudioJack2_SwitchT J?
-U 1 1 5D79954C
-P 4675 7000
-AR Path="/5CF11B19/5D79954C" Ref="J?"  Part="1"
-AR Path="/5D4DB615/5D79954C" Ref="J304"  Part="1"
-F 0 "J304" H 4442 7071 50  0000 R CNN
-F 1 "In 2" H 4442 6980 50  0000 R CNN
-F 2 "AJ-Dropbox-Kicad:PJ301SM" H 4675 7000 50  0001 C CNN
-F 3 "~" H 4675 7000 50  0001 C CNN
-F 4 "VC input" H 4675 7000 50  0001 C CNN "Function"
-	1    4675 7000
-	-1   0    0    -1
-$EndComp
-Wire Wire Line
-	4475 7100 4375 7100
-Wire Wire Line
-	4375 7100 4375 6550
-Connection ~ 4375 6550
-Wire Wire Line
-	4375 6550 4475 6550
-Wire Wire Line
-	4475 6650 4425 6650
-Wire Wire Line
-	4425 6650 4425 7000
-Connection ~ 4425 7000
-Wire Wire Line
-	4425 7000 4475 7000
+F 0 "#PWR0313" H 4800 7000 50  0001 C CNN
+F 1 "GND" H 4805 7077 50  0000 C CNN
+F 2 "" H 4800 7250 50  0001 C CNN
+F 3 "" H 4800 7250 50  0001 C CNN
+	1    4800 7250
+	1    0    0    -1
+$EndComp
 Text GLabel 3275 6550 0    50   Input ~ 0
-In_1
+In_L
 Text GLabel 3275 7000 0    50   Input ~ 0
-In_2
+In_R
 Wire Wire Line
 	3275 7000 3425 7000
@@
 	0    1    1    0
 $EndComp
-Wire Wire Line
-	3725 6550 3750 6550
 $Comp
 L Device:C C?
@@
 	0    1    1    0
 $EndComp
-Wire Wire Line
-	3725 7000 3750 7000
 $Comp
 L Connector:AudioJack2 J?
@@
 Out2_Final
 Connection ~ 5900 6525
-$Comp
-L Device:D_Zener D?
-U 1 1 5D799579
-P 3750 6700
-AR Path="/5CF11B19/5D799579" Ref="D?"  Part="1"
-AR Path="/5D4DB615/5D799579" Ref="D311"  Part="1"
-F 0 "D311" V 3704 6779 50  0000 L CNN
-F 1 "D_Zener" V 3795 6779 50  0000 L CNN
-F 2 "Diode_SMD:D_MiniMELF" H 3750 6700 50  0001 C CNN
-F 3 "~" H 3750 6700 50  0001 C CNN
-	1    3750 6700
-	0    1    1    0
-$EndComp
-Connection ~ 3750 6550
-Wire Wire Line
-	3750 6550 3875 6550
-$Comp
-L Device:D_Zener D?
-U 1 1 5D799581
-P 3750 7150
-AR Path="/5CF11B19/5D799581" Ref="D?"  Part="1"
-AR Path="/5D4DB615/5D799581" Ref="D312"  Part="1"
-F 0 "D312" V 3704 7229 50  0000 L CNN
-F 1 "D_Zener" V 3795 7229 50  0000 L CNN
-F 2 "Diode_SMD:D_MiniMELF" H 3750 7150 50  0001 C CNN
-F 3 "~" H 3750 7150 50  0001 C CNN
-	1    3750 7150
-	0    1    1    0
-$EndComp
-Connection ~ 3750 7000
-Wire Wire Line
-	3750 7000 3875 7000
-Wire Wire Line
-	3750 6850 3750 6900
-Wire Wire Line
-	3750 6900 4325 6900
-Wire Wire Line
-	4325 7150 4325 7300
-Wire Wire Line
-	3750 7300 4325 7300
-Connection ~ 4325 7300
-Wire Wire Line
-	4325 7300 4325 7350
 Wire Wire Line
 	1850 6575 2125 6575
@@
 	1    0    0    1
 $EndComp
-Text GLabel 3950 2450 0    50   Input ~ 0
-In_1
-Text GLabel 3925 4450 0    50   Input ~ 0
-In_2
 $Comp
 L Device:R R?
@@
 Wire Wire Line
 	4300 2250 4300 1950
-Wire Wire Line
-	5250 1950 5250 2000
 Wire Wire Line
 	5250 2350 5050 2350
@@
 Wire Notes Line
 	5100 5925 5100 7725
-Text HLabel 5175 4100 1    50   Input ~ 0
-POT3_H
-Text HLabel 5075 4100 1    50   Input ~ 0
-POT3_C
-Text HLabel 4975 4100 1    50   Input ~ 0
-POT3_L
 $Comp
 L Diode:LL4148 D?
@@
 Wire Wire Line
 	4550 4125 4625 4125
-Wire Wire Line
-	4975 4125 4975 4100
 Connection ~ 4550 4125
 Wire Wire Line
-	5075 4100 5075 4125
-Wire Wire Line
-	5075 4125 5175 4125
-Connection ~ 5275 4125
-Wire Wire Line
-	5275 4125 5275 4450
-Wire Wire Line
-	5175 4100 5175 4125
-Connection ~ 5175 4125
-Wire Wire Line
-	5175 4125 5275 4125
-Wire Wire Line
 	5275 3725 4950 3725
-Wire Wire Line
-	5275 3725 5275 4125
 Wire Wire Line
 	4150 3725 4150 3825
@@
 $EndComp
 Wire Wire Line
-	4925 4125 4975 4125
-Text HLabel 8200 3925 1    50   Input ~ 0
-POT4_H
-Text HLabel 8100 3925 1    50   Input ~ 0
-POT4_C
-Text HLabel 8000 3925 1    50   Input ~ 0
-POT4_L
-Wire Wire Line
 	8275 3925 8275 4550
 Wire Wire Line
@@
 Wire Wire Line
 	8875 4550 8925 4550
-Wire Wire Line
-	8100 3925 8275 3925
-Wire Wire Line
-	8000 3925 7900 3925
-Text HLabel 4900 1950 1    50   Input ~ 0
-POT1_H
-Text HLabel 4800 1950 1    50   Input ~ 0
-POT1_C
-Text HLabel 4700 1950 1    50   Input ~ 0
-POT1_L
-Wire Wire Line
-	4700 1950 4300 1950
-Wire Wire Line
-	4800 1950 5250 1950
-Text HLabel 7925 1950 1    50   Input ~ 0
-POT2_H
-Text HLabel 7825 1950 1    50   Input ~ 0
-POT2_C
-Text HLabel 7725 1950 1    50   Input ~ 0
-POT2_L
-Wire Wire Line
-	7725 1950 7400 1950
-Wire Wire Line
-	7825 1950 8300 1950
 $Comp
 L Device:R R?
@@
 Wire Wire Line
 	7275 1950 7400 1950
-Connection ~ 7400 1950
 $Comp
 L power:GND #PWR?
@@
 Wire Wire Line
 	5250 1475 5250 1575
-Connection ~ 5250 1950
 Wire Wire Line
 	4850 1075 4300 1075
@@
 	1    0    0    -1
 $EndComp
-Wire Wire Line
-	5250 1875 5250 1950
 $Comp
 L Diode:LL4148 D?
@@
 	3850 4125 4150 4125
 Connection ~ 4150 4125
+$Comp
+L Connector:Conn_Coaxial_x2 J?
+U 1 1 5DBB8503
+P 4800 6650
+F 0 "J?" H 4728 6988 50  0000 C CNN
+F 1 "Conn_Coaxial_x2" H 4728 6897 50  0000 C CNN
+F 2 "" H 4800 6550 50  0001 C CNN
+F 3 " ~" H 4800 6550 50  0001 C CNN
+	1    4800 6650
+	1    0    0    -1
+$EndComp
+Wire Wire Line
+	5275 3725 5275 4450
+Wire Wire Line
+	5250 1875 5250 2000
+Wire Wire Line
+	3725 6550 3875 6550
+Wire Wire Line
+	3725 7000 3875 7000
+Wire Wire Line
+	4800 6950 4800 7150
+Wire Wire Line
+	4600 6550 4225 6550
+Wire Wire Line
+	4225 7000 4600 7000
+Wire Wire Line
+	4600 7000 4600 6750
+Wire Wire Line
+	4225 6700 4450 6700
+Wire Wire Line
+	4450 6700 4450 7150
+Wire Wire Line
+	4450 7150 4800 7150
+Connection ~ 4800 7150
+Wire Wire Line
+	4800 7150 4800 7250
+Wire Wire Line
+	4225 7150 4450 7150
+Connection ~ 4450 7150
+Text GLabel 2825 3075 0    50   Input ~ 0
+In_L
+Text GLabel 2825 3525 0    50   Input ~ 0
+In_R
 $EndSCHEMATC

Commit message: RCA on RIAA
Parts:
- removed C305, C307, C313, C314: 1u, Capacitor_SMD:C_0805_2012Metric_Pad1.15x1.40mm_HandSolder, symbol Device:C
- removed J301: Out 1, AJ-Dropbox-Kicad:PJ301SM, symbol Connector:AudioJack2
- removed J303: Out 2, AJ-Dropbox-Kicad:PJ301SM, symbol Connector:AudioJack2
- removed J305: Out 1 Final, AJ-Dropbox-Kicad:PJ301SM, symbol Connector:AudioJack2
- removed J306: Out 2 Final, AJ-Dropbox-Kicad:PJ301SM, symbol Connector:AudioJack2
- added C? (x2): 1u, Capacitor_SMD:C_0805_2012Metric_Pad1.15x1.40mm_HandSolder, symbol Device:C
- added J?: Conn_Coaxial_x2, symbol Connector:Conn_Coaxial_x2
Connections:
- net labels added: Out_L, Out_R
- wire segments 155 -> 145
Changed lines of the file:
@@
 	2125 6575 2525 6575
-$Comp
-L Connector:AudioJack2 J?
-U 1 1 5D7994F9
-P 6250 6225
-AR Path="/5CF11B19/5D7994F9" Ref="J?"  Part="1"
-AR Path="/5D4DB615/5D7994F9" Ref="J301"  Part="1"
-F 0 "J301" H 6017 6296 50  0000 R CNN
-F 1 "Out 1" H 6017 6205 50  0000 R CNN
-F 2 "AJ-Dropbox-Kicad:PJ301SM" H 6250 6225 50  0001 C CNN
-F 3 "~" H 6250 6225 50  0001 C CNN
-	1    6250 6225
-	-1   0    0    -1
-$EndComp
-$Comp
-L Connector:AudioJack2 J?
-U 1 1 5D7994FF
-P 6250 6625
-AR Path="/5CF11B19/5D7994FF" Ref="J?"  Part="1"
-AR Path="/5D4DB615/5D7994FF" Ref="J303"  Part="1"
-F 0 "J303" H 6017 6696 50  0000 R CNN
-F 1 "Out 2" H 6017 6605 50  0000 R CNN
-F 2 "AJ-Dropbox-Kicad:PJ301SM" H 6250 6625 50  0001 C CNN
-F 3 "~" H 6250 6625 50  0001 C CNN
-	1    6250 6625
-	-1   0    0    -1
-$EndComp
-Wire Wire Line
-	6050 6125 5900 6125
-Wire Wire Line
-	6050 6525 5900 6525
 $Comp
 L Device:R R?
@@
 	0    -1   -1   0
 $EndComp
-Wire Wire Line
-	5900 6125 5900 6525
 Connection ~ 3875 6550
 Wire Wire Line
@@
 $Comp
 L power:GND #PWR?
-U 1 1 5D79953C
-P 5900 7475
-AR Path="/5CF11B19/5D79953C" Ref="#PWR?"  Part="1"
-AR Path="/5D4DB615/5D79953C" Ref="#PWR0314"  Part="1"
-F 0 "#PWR0314" H 5900 7225 50  0001 C CNN
-F 1 "GND" H 5905 7302 50  0000 C CNN
-F 2 "" H 5900 7475 50  0001 C CNN
-F 3 "" H 5900 7475 50  0001 C CNN
-	1    5900 7475
-	1    0    0    -1
-$EndComp
-Text GLabel 5525 6625 0    50   Input ~ 0
-Out2_Dist
-Text GLabel 5525 6225 0    50   Input ~ 0
-Out1_Dist
-$Comp
-L power:GND #PWR?
 U 1 1 5D799544
 P 4800 7250
@@
 	0    1    1    0
 $EndComp
-$Comp
-L Connector:AudioJack2 J?
-U 1 1 5D79956C
-P 6250 7375
-AR Path="/5CF11B19/5D79956C" Ref="J?"  Part="1"
-AR Path="/5D4DB615/5D79956C" Ref="J306"  Part="1"
-F 0 "J306" H 6017 7446 50  0000 R CNN
-F 1 "Out 2 Final" H 6017 7355 50  0000 R CNN
-F 2 "AJ-Dropbox-Kicad:PJ301SM" H 6250 7375 50  0001 C CNN
-F 3 "~" H 6250 7375 50  0001 C CNN
-	1    6250 7375
-	-1   0    0    -1
-$EndComp
-Wire Wire Line
-	6050 7275 5900 7275
-Wire Wire Line
-	5900 7475 5900 7275
-Wire Wire Line
-	5900 6525 5900 6925
-Text GLabel 5525 7375 0    50   Input ~ 0
-Out2_Final
-Connection ~ 5900 6525
 Wire Wire Line
 	1850 6575 2125 6575
@@
 Wire Wire Line
 	8125 4550 8275 4550
-$Comp
-L Connector:AudioJack2 J?
-U 1 1 5D84994A
-P 6250 7025
-AR Path="/5CF11B19/5D84994A" Ref="J?"  Part="1"
-AR Path="/5D4DB615/5D84994A" Ref="J305"  Part="1"
-F 0 "J305" H 6017 7096 50  0000 R CNN
-F 1 "Out 1 Final" H 6017 7005 50  0000 R CNN
-F 2 "AJ-Dropbox-Kicad:PJ301SM" H 6250 7025 50  0001 C CNN
-F 3 "~" H 6250 7025 50  0001 C CNN
-	1    6250 7025
-	-1   0    0    -1
-$EndComp
-Text GLabel 5525 7025 0    50   Input ~ 0
-Out1_Final
-Wire Wire Line
-	6050 6925 5900 6925
-Wire Wire Line
-	5900 7275 5900 6925
-Connection ~ 5900 7275
-Connection ~ 5900 6925
 Text GLabel 8975 4550 2    50   Input ~ 0
 Out2_Final
@@
 Wire Wire Line
 	6775 4875 6775 4950
-$Comp
-L Device:C C?
-U 1 1 5D8781E6
-P 5725 6225
-AR Path="/5CF11B19/5D8781E6" Ref="C?"  Part="1"
-AR Path="/5D4DB615/5D8781E6" Ref="C305"  Part="1"
-F 0 "C305" V 5875 6175 50  0000 L CNN
-F 1 "1u" V 5575 6150 50  0000 L CNN
-F 2 "Capacitor_SMD:C_0805_2012Metric_Pad1.15x1.40mm_HandSolder" H 5763 6075 50  0001 C CNN
-F 3 "~" H 5725 6225 50  0001 C CNN
-	1    5725 6225
-	0    1    1    0
-$EndComp
-Wire Wire Line
-	5525 6225 5575 6225
-Wire Wire Line
-	5525 6625 5575 6625
-Wire Wire Line
-	5525 7025 5575 7025
-Wire Wire Line
-	5525 7375 5575 7375
-Wire Wire Line
-	5875 6225 6050 6225
-$Comp
-L Device:C C?
-U 1 1 5D88B3A1
-P 5725 6625
-AR Path="/5CF11B19/5D88B3A1" Ref="C?"  Part="1"
-AR Path="/5D4DB615/5D88B3A1" Ref="C307"  Part="1"
-F 0 "C307" V 5875 6575 50  0000 L CNN
-F 1 "1u" V 5575 6550 50  0000 L CNN
-F 2 "Capacitor_SMD:C_0805_2012Metric_Pad1.15x1.40mm_HandSolder" H 5763 6475 50  0001 C CNN
-F 3 "~" H 5725 6625 50  0001 C CNN
-	1    5725 6625
-	0    1    1    0
-$EndComp
-Wire Wire Line
-	5875 6625 6050 6625
-$Comp
-L Device:C C?
-U 1 1 5D88B72B
-P 5725 7025
-AR Path="/5CF11B19/5D88B72B" Ref="C?"  Part="1"
-AR Path="/5D4DB615/5D88B72B" Ref="C313"  Part="1"
-F 0 "C313" V 5875 6975 50  0000 L CNN
-F 1 "1u" V 5575 6950 50  0000 L CNN
-F 2 "Capacitor_SMD:C_0805_2012Metric_Pad1.15x1.40mm_HandSolder" H 5763 6875 50  0001 C CNN
-F 3 "~" H 5725 7025 50  0001 C CNN
-	1    5725 7025
-	0    1    1    0
-$EndComp
-Wire Wire Line
-	5875 7025 6050 7025
-$Comp
-L Device:C C?
-U 1 1 5D88BB07
-P 5725 7375
-AR Path="/5CF11B19/5D88BB07" Ref="C?"  Part="1"
-AR Path="/5D4DB615/5D88BB07" Ref="C314"  Part="1"
-F 0 "C314" V 5875 7325 50  0000 L CNN
-F 1 "1u" V 5575 7300 50  0000 L CNN
-F 2 "Capacitor_SMD:C_0805_2012Metric_Pad1.15x1.40mm_HandSolder" H 5763 7225 50  0001 C CNN
-F 3 "~" H 5725 7375 50  0001 C CNN
-	1    5725 7375
-	0    1    1    0
-$EndComp
-Wire Wire Line
-	5875 7375 6050 7375
 $Comp
 L power:GND #PWR?
@@
 Text GLabel 2825 3525 0    50   Input ~ 0
 In_R
+$Comp
+L power:GND #PWR?
+U 1 1 5DC3A5B0
+P 6500 7250
+AR Path="/5CF11B19/5DC3A5B0" Ref="#PWR?"  Part="1"
+AR Path="/5D4DB615/5DC3A5B0" Ref="#PWR?"  Part="1"
+F 0 "#PWR?" H 6500 7000 50  0001 C CNN
+F 1 "GND" H 6505 7077 50  0000 C CNN
+F 2 "" H 6500 7250 50  0001 C CNN
+F 3 "" H 6500 7250 50  0001 C CNN
+	1    6500 7250
+	1    0    0    -1
+$EndComp
+Text GLabel 5750 6550 0    50   Input ~ 0
+Out_L
+Text GLabel 5750 7000 0    50   Input ~ 0
+Out_R
+Wire Wire Line
+	5750 7000 5900 7000
+Wire Wire Line
+	5750 6550 5900 6550
+$Comp
+L Device:C C?
+U 1 1 5DC3A5BE
+P 6050 6550
+AR Path="/5CF11B19/5DC3A5BE" Ref="C?"  Part="1"
+AR Path="/5D4DB615/5DC3A5BE" Ref="C?"  Part="1"
+F 0 "C?" V 6200 6500 50  0000 L CNN
+F 1 "1u" V 5900 6475 50  0000 L CNN
+F 2 "Capacitor_SMD:C_0805_2012Metric_Pad1.15x1.40mm_HandSolder" H 6088 6400 50  0001 C CNN
+F 3 "~" H 6050 6550 50  0001 C CNN
+	1    6050 6550
+	0    1    1    0
+$EndComp
+$Comp
+L Device:C C?
+U 1 1 5DC3A5C8
+P 6050 7000
+AR Path="/5CF11B19/5DC3A5C8" Ref="C?"  Part="1"
+AR Path="/5D4DB615/5DC3A5C8" Ref="C?"  Part="1"
+F 0 "C?" V 6200 6950 50  0000 L CNN
+F 1 "1u" V 5900 6925 50  0000 L CNN
+F 2 "Capacitor_SMD:C_0805_2012Metric_Pad1.15x1.40mm_HandSolder" H 6088 6850 50  0001 C CNN
+F 3 "~" H 6050 7000 50  0001 C CNN
+	1    6050 7000
+	0    1    1    0
+$EndComp
+$Comp
+L Connector:Conn_Coaxial_x2 J?
+U 1 1 5DC3A5D2
+P 6500 6650
+F 0 "J?" H 6428 6988 50  0000 C CNN
+F 1 "Conn_Coaxial_x2" H 6428 6897 50  0000 C CNN
+F 2 "" H 6500 6550 50  0001 C CNN
+F 3 " ~" H 6500 6550 50  0001 C CNN
+	1    6500 6650
+	1    0    0    -1
+$EndComp
+Wire Wire Line
+	6300 7000 6300 6750
+Wire Wire Line
+	6500 6950 6500 7250
+Wire Wire Line
+	6200 6550 6300 6550
+Wire Wire Line
+	6300 7000 6200 7000
 $EndSCHEMATC
