File: KicadJE_AteOhAte/KicadJE_AteOhAte3.sch (KiCad schematic (older format))
At the start: 84 parts, among them J301 PJRAS2X2S01AUX, U301 TL072, U302 TL072, U303 TL072

Commit message: PWR RIAA
Parts:
- removed D301, D302: LL4148, Diode_SMD:D_MiniMELF, symbol Diode:LL4148
- removed D303: LED, LED_THT:LED_D3.0mm, symbol Device:LED
- added C345, C346: 470u, Capacitor_THT:CP_Radial_D13.0mm_P5.00mm, symbol Device:CP
- added J302: Conn_01x03, TerminalBlock:TerminalBlock_bornier-3_P5.08mm, symbol Connector_Generic:Conn_01x03
- added R329, R330: 1R1, Resistor_SMD:R_0805_2012Metric_Pad1.15x1.40mm_HandSolder, symbol Device:R
Connections:
- net +12V: now also C345.1, R329.1
- net -12V: now also C346.2, R330.1
- net GND: now also C345.2, C346.1, J302.2 (Pin_2)
- net at D304.1 (K): now also J302.1 (Pin_1), R330.2
- net at R327.2: now also J302.3 (Pin_3), R329.2
Other:
- moved on the sheet: D304, R327
Changed lines of the file:
@@
 AR Path="/5D4DB615/5D5139E9" Ref="#FLG0302"  Part="1"
 F 0 "#FLG0302" H 1500 6950 50  0001 C CNN
-F 1 "PWR_FLAG" H 1500 7049 50  0000 C CNN
+F 1 "PWR_FLAG" H 1425 6875 50  0000 C CNN
 F 2 "" H 1500 6875 50  0001 C CNN
 F 3 "~" H 1500 6875 50  0001 C CNN
@@
 AR Path="/5D4DB615/5D513A1F" Ref="#FLG0303"  Part="1"
 F 0 "#FLG0303" H 1925 7250 50  0001 C CNN
-F 1 "PWR_FLAG" H 1925 7349 50  0000 C CNN
+F 1 "PWR_FLAG" H 1975 7175 50  0000 C CNN
 F 2 "" H 1925 7175 50  0001 C CNN
 F 3 "~" H 1925 7175 50  0001 C CNN
@@
 	7300 1900 6975 1900
 $Comp
-L Diode:LL4148 D?
-U 1 1 5D90A096
-P 1875 2025
-AR Path="/5CF11B19/5D90A096" Ref="D?"  Part="1"
-AR Path="/5D4DB615/5D90A096" Ref="D302"  Part="1"
-F 0 "D302" V 2075 1825 50  0000 L CNN
-F 1 "LL4148" V 1650 1850 50  0000 L CNN
-F 2 "Diode_SMD:D_MiniMELF" H 1875 1850 50  0001 C CNN
-F 3 "http://www.vishay.com/docs/85557/ll4148.pdf" H 1875 2025 50  0001 C CNN
-	1    1875 2025
-	0    -1   -1   0
-$EndComp
-$Comp
-L Diode:LL4148 D?
-U 1 1 5D90A0A0
-P 1700 2025
-AR Path="/5CF11B19/5D90A0A0" Ref="D?"  Part="1"
-AR Path="/5D4DB615/5D90A0A0" Ref="D301"  Part="1"
-F 0 "D301" V 1475 2050 50  0000 R CNN
-F 1 "LL4148" V 1700 1975 50  0000 R CNN
-F 2 "Diode_SMD:D_MiniMELF" H 1700 1850 50  0001 C CNN
-F 3 "http://www.vishay.com/docs/85557/ll4148.pdf" H 1700 2025 50  0001 C CNN
-	1    1700 2025
-	0    1    1    0
-$EndComp
-$Comp
 L Device:R R?
 U 1 1 5D9D0730
@@
 L Device:LED D304
 U 1 1 5DA59B0A
-P 775 5500
-F 0 "D304" V 814 5382 50  0000 R CNN
-F 1 "LED" V 723 5382 50  0000 R CNN
-F 2 "LED_THT:LED_D3.0mm" H 775 5500 50  0001 C CNN
-F 3 "~" H 775 5500 50  0001 C CNN
-	1    775  5500
+P 1025 7025
+F 0 "D304" V 1100 7125 50  0000 R CNN
+F 1 "LED" V 1000 7225 50  0000 R CNN
+F 2 "LED_THT:LED_D3.0mm" H 1025 7025 50  0001 C CNN
+F 3 "~" H 1025 7025 50  0001 C CNN
+	1    1025 7025
 	0    -1   -1   0
 $EndComp
@@
 L Device:R R?
 U 1 1 5DA66984
-P 775 5200
+P 1025 6725
 AR Path="/5CF11B19/5DA66984" Ref="R?"  Part="1"
 AR Path="/5D4DB615/5DA66984" Ref="R327"  Part="1"
-F 0 "R327" V 875 5175 50  0000 C CNN
-F 1 "12k" V 700 5300 50  0000 C CNN
-F 2 "Resistor_SMD:R_0805_2012Metric_Pad1.15x1.40mm_HandSolder" V 705 5200 50  0001 C CNN
-F 3 "~" H 775 5200 50  0001 C CNN
-	1    775  5200
+F 0 "R327" V 1125 6700 50  0000 C CNN
+F 1 "12k" V 950 6825 50  0000 C CNN
+F 2 "Resistor_SMD:R_0805_2012Metric_Pad1.15x1.40mm_HandSolder" V 955 6725 50  0001 C CNN
+F 3 "~" H 1025 6725 50  0001 C CNN
+	1    1025 6725
 	-1   0    0    1
-$EndComp
-$Comp
-L Device:LED D303
-U 1 1 5DB1DBA3
-P 1225 2050
-F 0 "D303" V 1264 1932 50  0000 R CNN
-F 1 "LED" V 1173 1932 50  0000 R CNN
-F 2 "LED_THT:LED_D3.0mm" H 1225 2050 50  0001 C CNN
-F 3 "~" H 1225 2050 50  0001 C CNN
-	1    1225 2050
-	0    -1   -1   0
 $EndComp
 Wire Wire Line
@@
 Wire Wire Line
 	2250 7175 2525 7175
+$Comp
+L Connector_Generic:Conn_01x03 J302
+U 1 1 5E1DC818
+P 700 6875
+F 0 "J302" H 618 6550 50  0000 C CNN
+F 1 "Conn_01x03" H 618 6641 50  0000 C CNN
+F 2 "TerminalBlock:TerminalBlock_bornier-3_P5.08mm" H 700 6875 50  0001 C CNN
+F 3 "~" H 700 6875 50  0001 C CNN
+	1    700  6875
+	-1   0    0    1
+$EndComp
+Connection ~ 1500 6875
+Wire Wire Line
+	900  6975 900  7175
+Wire Wire Line
+	900  7175 1025 7175
+Connection ~ 1700 7175
+Wire Wire Line
+	900  6775 900  6575
+Wire Wire Line
+	900  6575 1025 6575
+Connection ~ 1700 6575
+Connection ~ 1025 6575
+Connection ~ 1025 7175
+$Comp
+L Device:CP C345
+U 1 1 5E21B81B
+P 1400 6725
+F 0 "C345" H 1450 6800 50  0000 C CNN
+F 1 "470u" H 1275 6625 50  0000 C CNN
+F 2 "Capacitor_THT:CP_Radial_D13.0mm_P5.00mm" H 1438 6575 50  0001 C CNN
+F 3 "~" H 1400 6725 50  0001 C CNN
+	1    1400 6725
+	1    0    0    -1
+$EndComp
+$Comp
+L Device:CP C346
+U 1 1 5E21C344
+P 1400 7025
+F 0 "C346" H 1250 7125 50  0000 C CNN
+F 1 "470u" H 1200 7025 50  0000 C CNN
+F 2 "Capacitor_THT:CP_Radial_D13.0mm_P5.00mm" H 1438 6875 50  0001 C CNN
+F 3 "~" H 1400 7025 50  0001 C CNN
+	1    1400 7025
+	1    0    0    -1
+$EndComp
+$Comp
+L Device:R R?
+U 1 1 5E21C9CA
+P 1225 6575
+AR Path="/5CF11B19/5E21C9CA" Ref="R?"  Part="1"
+AR Path="/5D4DB615/5E21C9CA" Ref="R329"  Part="1"
+F 0 "R329" V 1325 6550 50  0000 C CNN
+F 1 "1R1" V 1225 6575 50  0000 C CNN
+F 2 "Resistor_SMD:R_0805_2012Metric_Pad1.15x1.40mm_HandSolder" V 1155 6575 50  0001 C CNN
+F 3 "~" H 1225 6575 50  0001 C CNN
+	1    1225 6575
+	0    1    1    0
+$EndComp
+$Comp
+L Device:R R?
+U 1 1 5E21D2E2
+P 1225 7175
+AR Path="/5CF11B19/5E21D2E2" Ref="R?"  Part="1"
+AR Path="/5D4DB615/5E21D2E2" Ref="R330"  Part="1"
+F 0 "R330" V 1325 7150 50  0000 C CNN
+F 1 "1R1" V 1225 7150 50  0000 C CNN
+F 2 "Resistor_SMD:R_0805_2012Metric_Pad1.15x1.40mm_HandSolder" V 1155 7175 50  0001 C CNN
+F 3 "~" H 1225 7175 50  0001 C CNN
+	1    1225 7175
+	0    1    1    0
+$EndComp
+Connection ~ 1400 6875
+Wire Wire Line
+	1400 6875 1500 6875
+Connection ~ 1400 7175
+Wire Wire Line
+	1400 7175 1700 7175
+Connection ~ 1400 6575
+Wire Wire Line
+	1400 6575 1700 6575
+Wire Wire Line
+	1025 7175 1075 7175
+Wire Wire Line
+	900  6875 1400 6875
+Wire Wire Line
+	1025 6575 1075 6575
+Wire Wire Line
+	1375 7175 1400 7175
+Wire Wire Line
+	1375 6575 1400 6575
 $EndSCHEMATC
