File: KicadJE_AteOhAte - RevB/KicadJE_AteOhAte2.sch (KiCad schematic (older format))
At the start: 113 parts, among them J201 In_Accent, J202 In Gate, J203 Out Tom, P201 Doepfer_Power_10pin, Q201 MMBT2222A, Q202 MMBT2222A, Q203 MMBT2222A, Q204 MMBT2222A, Q205 MMBT2907A, Q206 MMBT2222A, Q207 MMBT2222A, SW201 Con/Tom, U201 TL072, U202 TL072, U203 TL072

Commit message: New tom ext noise
Parts:
- removed C201, C202, C203, C204: 100n, Capacitor_SMD:C_0805_2012Metric_Pad1.15x1.40mm_HandSolder, symbol Device:C
- removed C205: 39n, Capacitor_SMD:C_0805_2012Metric_Pad1.15x1.40mm_HandSolder, symbol Device:C
- removed C206: 1u, Capacitor_SMD:C_0805_2012Metric_Pad1.15x1.40mm_HandSolder, symbol Device:C
- removed C207: 22u, Capacitor_SMD:C_0805_2012Metric_Pad1.15x1.40mm_HandSolder, symbol Device:C
- removed C208: 18n, Capacitor_SMD:C_0805_2012Metric_Pad1.15x1.40mm_HandSolder, symbol Device:C
- removed C209: C11, Capacitor_SMD:C_0805_2012Metric_Pad1.15x1.40mm_HandSolder, symbol Device:C
- removed C210: C9, Capacitor_SMD:C_0805_2012Metric_Pad1.15x1.40mm_HandSolder, symbol Device:C
- removed C211: C10, Capacitor_SMD:C_0805_2012Metric_Pad1.15x1.40mm_HandSolder, symbol Device:C
- removed C212: 1n, Capacitor_SMD:C_0805_2012Metric_Pad1.15x1.40mm_HandSolder, symbol Device:C
- removed C213: C12, Capacitor_SMD:C_0805_2012Metric_Pad1.15x1.40mm_HandSolder, symbol Device:C
- removed C214: C8, Capacitor_SMD:C_0805_2012Metric_Pad1.15x1.40mm_HandSolder, symbol Device:C
- removed C215: C6, Capacitor_SMD:C_0805_2012Metric_Pad1.15x1.40mm_HandSolder, symbol Device:C
- removed C216: 47n, Capacitor_SMD:C_0805_2012Metric_Pad1.15x1.40mm_HandSolder, symbol Device:C
- removed C217: 10n, Capacitor_SMD:C_0805_2012Metric_Pad1.15x1.40mm_HandSolder, symbol Device:C
- removed C218: C7, Capacitor_SMD:C_0805_2012Metric_Pad1.15x1.40mm_HandSolder, symbol Device:C
- removed C219: C4, Capacitor_SMD:C_0805_2012Metric_Pad1.15x1.40mm_HandSolder, symbol Device:C
- removed C220, C221: 10u, Capacitor_SMD:C_1206_3216Metric_Pad1.42x1.75mm_HandSolder, symbol Device:C
- removed D201, D202: 1N1007, Diode_SMD:D_SOD-123, symbol Device:D
- removed D203, D204: D_Zener, Diode_SMD:D_MiniMELF, symbol Device:D_Zener
- removed D205, D206, D207, D208, D209: 1N4148, Diode_SMD:D_SOD-123, symbol Device:D
- removed H201, H202: 2,5mm, MountingHole:MountingHole_2.5mm_Pad_Via, symbol Mechanical:MountingHole
- removed H203, H204: 2,2mm, MountingHole:MountingHole_2.2mm_M2_Pad_Via, symbol Mechanical:MountingHole
- removed J201: In_Accent, Connector_Audio:Jack_3.5mm_Ledino_KB3SPRS_Horizontal, symbol Connector:AudioJack2_SwitchT
- removed J202: In Gate, AJ-Dropbox-Kicad:PJ301SM, symbol Connector:AudioJack2_SwitchT
- removed J203: Out Tom, AJ-Dropbox-Kicad:PJ301SM, symbol Connector:AudioJack2
- removed JP201: Jumper, Connector_PinHeader_2.54mm:PinHeader_1x02_P2.54mm_Vertical, symbol Device:Jumper
- removed P201: Doepfer_Power_10pin, Connectors_IDC:IDC-Header_2x05_Pitch2.54mm_Straight, symbol Eurorack:Doepfer_Power_10pin
- removed Q201, Q202, Q203, Q204, Q206, Q207: MMBT2222A, Package_TO_SOT_SMD:SOT-23_Handsoldering, symbol MMBT2222A:MMBT2222A
- removed Q205: MMBT2907A, Package_TO_SOT_SMD:SOT-23_Handsoldering, symbol MMBT2907_:MMBT2907*
- removed R201, R206: 1M, Resistor_SMD:R_0805_2012Metric_Pad1.15x1.40mm_HandSolder, symbol Device:R
- removed R202, R220, R221, R228, R229, R233, R235, R238, R239, R242: 4k7, Resistor_SMD:R_0805_2012Metric_Pad1.15x1.40mm_HandSolder, symbol Device:R
- removed R203: 330K, Resistor_SMD:R_0805_2012Metric_Pad1.15x1.40mm_HandSolder, symbol Device:R
- removed R204: 100R, Resistor_SMD:R_0805_2012Metric_Pad1.15x1.40mm_HandSolder, symbol Device:R
- removed R205, R207, R232, R240, R241, R245, R250: 22k, Resistor_SMD:R_0805_2012Metric_Pad1.15x1.40mm_HandSolder, symbol Device:R
- removed R208: 300R, Resistor_SMD:R_0805_2012Metric_Pad1.15x1.40mm_HandSolder, symbol Device:R
- removed R209, R211: 1K, Resistor_SMD:R_0805_2012Metric_Pad1.15x1.40mm_HandSolder, symbol Device:R
- removed R210, R213: OPEN, Resistor_SMD:R_0805_2012Metric_Pad1.15x1.40mm_HandSolder, symbol Device:R
- removed R212: 0R, Resistor_SMD:R_0805_2012Metric_Pad1.15x1.40mm_HandSolder, symbol Device:R
- removed R214, R225: 1k, Resistor_SMD:R_0805_2012Metric_Pad1.15x1.40mm_HandSolder, symbol Device:R
- removed R215, R222: 470k, Resistor_SMD:R_0805_2012Metric_Pad1.15x1.40mm_HandSolder, symbol Device:R
- removed R216: 820k, Resistor_SMD:R_0805_2012Metric_Pad1.15x1.40mm_HandSolder, symbol Device:R
- removed R217, R223, R244, R249: 33k, Resistor_SMD:R_0805_2012Metric_Pad1.15x1.40mm_HandSolder, symbol Device:R
- removed R218, R219, R224, R234, R251, R252, R253, R254: 100k, Resistor_SMD:R_0805_2012Metric_Pad1.15x1.40mm_HandSolder, symbol Device:R
- removed R226: 15k, Resistor_SMD:R_0805_2012Metric_Pad1.15x1.40mm_HandSolder, symbol Device:R
- removed R227, R236, R237, R246: 10k, Resistor_SMD:R_0805_2012Metric_Pad1.15x1.40mm_HandSolder, symbol Device:R
- removed R230: R17, Resistor_SMD:R_0805_2012Metric_Pad1.15x1.40mm_HandSolder, symbol Device:R
- removed R231: R18, Resistor_SMD:R_0805_2012Metric_Pad1.15x1.40mm_HandSolder, symbol Device:R
- removed R243: 3k3, Resistor_SMD:R_0805_2012Metric_Pad1.15x1.40mm_HandSolder, symbol Device:R
- removed R247: 47k, Resistor_SMD:R_0805_2012Metric_Pad1.15x1.40mm_HandSolder, symbol Device:R
- removed R248: 2M2, Resistor_SMD:R_0805_2012Metric_Pad1.15x1.40mm_HandSolder, symbol Device:R
- removed RV201: 100K, Potentiometer_THT:Potentiometer_Bourns_3296W_Vertical, symbol Device:R_POT_TRIM
- removed RV202: 50K, Potentiometer_THT:Potentiometer_Bourns_3296W_Vertical, symbol Device:R_POT_TRIM
- removed RV203: 500R Tune, Potentiometer_THT:Potentiometer_Piher_T-16H_Single_Horizontal, symbol Device:R_POT
- removed RV204: 1M Decay, Potentiometer_THT:Potentiometer_Piher_T-16H_Single_Horizontal, symbol Device:R_POT
- removed RV205: 100k A Level, Potentiometer_THT:Potentiometer_Piher_T-16H_Single_Horizontal, symbol Device:R_POT
- removed RV206: 100k A Reverb, Potentiometer_THT:Potentiometer_Piher_T-16H_Single_Horizontal, symbol Device:R_POT
- removed SW201: Con/Tom, AJ-Dropbox-Kicad:SPDTx2, symbol Switch:SW_DPDT_x2
- removed TP201: WhiteNoise, TestPoint:TestPoint_Pad_1.5x1.5mm, symbol Connector:TestPoint
- removed TP202: GND, TestPoint:TestPoint_THTPad_2.0x2.0mm_Drill1.0mm, symbol Connector:TestPoint
- removed TP203: Coupling, TestPoint:TestPoint_Pad_1.5x1.5mm, symbol Connector:TestPoint
- removed U201, U202, U203: TL072, AJ-Dropbox-Kicad:AJ_SO-8_5.3x6.2mm_P1.27mm, symbol Amplifier_Operational:TL072
- added C? (x4): 100n, Capacitor_SMD:C_0805_2012Metric_Pad1.15x1.40mm_HandSolder, symbol Device:C
- added C?: 10n, Capacitor_SMD:C_0805_2012Metric_Pad1.15x1.40mm_HandSolder, symbol Device:C
- added C?: C4, Capacitor_SMD:C_0805_2012Metric_Pad1.15x1.40mm_HandSolder, symbol Device:C
- added C?: C6, Capacitor_SMD:C_0805_2012Metric_Pad1.15x1.40mm_HandSolder, symbol Device:C
- added C?: C8, Capacitor_SMD:C_0805_2012Metric_Pad1.15x1.40mm_HandSolder, symbol Device:C
- added C?: C9, Capacitor_SMD:C_0805_2012Metric_Pad1.15x1.40mm_HandSolder, symbol Device:C
- added C?: C10, Capacitor_SMD:C_0805_2012Metric_Pad1.15x1.40mm_HandSolder, symbol Device:C
- added C?: C11, Capacitor_SMD:C_0805_2012Metric_Pad1.15x1.40mm_HandSolder, symbol Device:C
- added C?: C12, Capacitor_SMD:C_0805_2012Metric_Pad1.15x1.40mm_HandSolder, symbol Device:C
- added C?: 1n, Capacitor_SMD:C_0805_2012Metric_Pad1.15x1.40mm_HandSolder, symbol Device:C
- added C?: C7, Capacitor_SMD:C_0805_2012Metric_Pad1.15x1.40mm_HandSolder, symbol Device:C
- added C?: 47n, Capacitor_SMD:C_0805_2012Metric_Pad1.15x1.40mm_HandSolder, symbol Device:C
- added C?: 22u, Capacitor_SMD:C_0805_2012Metric_Pad1.15x1.40mm_HandSolder, symbol Device:C
- added C?: 1u, Capacitor_SMD:C_0805_2012Metric_Pad1.15x1.40mm_HandSolder, symbol Device:C
- added C?: 39n, Capacitor_SMD:C_0805_2012Metric_Pad1.15x1.40mm_HandSolder, symbol Device:C
- added C?: 18n, Capacitor_SMD:C_0805_2012Metric_Pad1.15x1.40mm_HandSolder, symbol Device:C
- added C? (x2): 10u, Capacitor_SMD:C_1206_3216Metric_Pad1.42x1.75mm_HandSolder, symbol Device:C
- added D? (x2): 1N1007, Diode_SMD:D_SOD-123, symbol Device:D
- added D? (x5): 1N4148, Diode_SMD:D_SOD-123, symbol Device:D
- added D? (x2): D_Zener, Diode_SMD:D_MiniMELF, symbol Device:D_Zener
- added H? (x2): 2,5mm, MountingHole:MountingHole_2.5mm_Pad_Via, symbol Mechanical:MountingHole
- added H? (x2): 2,2mm, MountingHole:MountingHole_2.2mm_M2_Pad_Via, symbol Mechanical:MountingHole
- added J?: In Gate, AJ-Dropbox-Kicad:PJ301SM, symbol Connector:AudioJack2_SwitchT
- added J?: Out Tom, AJ-Dropbox-Kicad:PJ301SM, symbol Connector:AudioJack2
- added J?: In_Accent, Connector_Audio:Jack_3.5mm_Ledino_KB3SPRS_Horizontal, symbol Connector:AudioJack2_SwitchT
- added JP?: Jumper, Connector_PinHeader_2.54mm:PinHeader_1x02_P2.54mm_Vertical, symbol Device:Jumper
- added P?: Doepfer_Power_10pin, Connectors_IDC:IDC-Header_2x05_Pitch2.54mm_Straight, symbol Eurorack:Doepfer_Power_10pin
- added Q? (x6): MMBT2222A, Package_TO_SOT_SMD:SOT-23_Handsoldering, symbol MMBT2222A:MMBT2222A
- added Q?: MMBT2907A, Package_TO_SOT_SMD:SOT-23_Handsoldering, symbol MMBT2907_:MMBT2907*
- added R? (x10): 4k7, Resistor_SMD:R_0805_2012Metric_Pad1.15x1.40mm_HandSolder, symbol Device:R
- added R? (x8): 100k, Resistor_SMD:R_0805_2012Metric_Pad1.15x1.40mm_HandSolder, symbol Device:R
- added R?: 47k, Resistor_SMD:R_0805_2012Metric_Pad1.15x1.40mm_HandSolder, symbol Device:R
- added R? (x4): 10k, Resistor_SMD:R_0805_2012Metric_Pad1.15x1.40mm_HandSolder, symbol Device:R
- added R?: 15k, Resistor_SMD:R_0805_2012Metric_Pad1.15x1.40mm_HandSolder, symbol Device:R
- added R? (x7): 22k, Resistor_SMD:R_0805_2012Metric_Pad1.15x1.40mm_HandSolder, symbol Device:R
- added R?: 2M2, Resistor_SMD:R_0805_2012Metric_Pad1.15x1.40mm_HandSolder, symbol Device:R
- added R? (x4): 33k, Resistor_SMD:R_0805_2012Metric_Pad1.15x1.40mm_HandSolder, symbol Device:R
- added R?: R17, Resistor_SMD:R_0805_2012Metric_Pad1.15x1.40mm_HandSolder, symbol Device:R
- added R?: R18, Resistor_SMD:R_0805_2012Metric_Pad1.15x1.40mm_HandSolder, symbol Device:R
- added R?: 820k, Resistor_SMD:R_0805_2012Metric_Pad1.15x1.40mm_HandSolder, symbol Device:R
- added R? (x2): 470k, Resistor_SMD:R_0805_2012Metric_Pad1.15x1.40mm_HandSolder, symbol Device:R
- added R? (x2): 1k, Resistor_SMD:R_0805_2012Metric_Pad1.15x1.40mm_HandSolder, symbol Device:R
- added R? (x2): 1K, Resistor_SMD:R_0805_2012Metric_Pad1.15x1.40mm_HandSolder, symbol Device:R
- added R? (x2): OPEN, Resistor_SMD:R_0805_2012Metric_Pad1.15x1.40mm_HandSolder, symbol Device:R
- added R?: 0R, Resistor_SMD:R_0805_2012Metric_Pad1.15x1.40mm_HandSolder, symbol Device:R
- added R?: 3k3, Resistor_SMD:R_0805_2012Metric_Pad1.15x1.40mm_HandSolder, symbol Device:R
- added R?: 100R, Resistor_SMD:R_0805_2012Metric_Pad1.15x1.40mm_HandSolder, symbol Device:R
- added R? (x2): 1M, Resistor_SMD:R_0805_2012Metric_Pad1.15x1.40mm_HandSolder, symbol Device:R
- added R?: 300R, Resistor_SMD:R_0805_2012Metric_Pad1.15x1.40mm_HandSolder, symbol Device:R
- added R?: 330K, Resistor_SMD:R_0805_2012Metric_Pad1.15x1.40mm_HandSolder, symbol Device:R
- added RV?: 1M Decay, Potentiometer_THT:Potentiometer_Piher_T-16H_Single_Horizontal, symbol Device:R_POT
- added RV?: 500R Tune, Potentiometer_THT:Potentiometer_Piher_T-16H_Single_Horizontal, symbol Device:R_POT
- added RV?: 100k A Reverb, Potentiometer_THT:Potentiometer_Piher_T-16H_Single_Horizontal, symbol Device:R_POT
- added RV?: 100k A Level, Potentiometer_THT:Potentiometer_Piher_T-16H_Single_Horizontal, symbol Device:R_POT
- added RV?: 100K, Potentiometer_THT:Potentiometer_Bourns_3296W_Vertical, symbol Device:R_POT_TRIM
- added RV?: 50K, Potentiometer_THT:Potentiometer_Bourns_3296W_Vertical, symbol Device:R_POT_TRIM
- added SW? (x2): Con/Tom, AJ-Dropbox-Kicad:SPDTx2, symbol Switch:SW_DPDT_x2
- added TP?: WhiteNoise, TestPoint:TestPoint_Pad_1.5x1.5mm, symbol Connector:TestPoint
- added TP?: GND, TestPoint:TestPoint_THTPad_2.0x2.0mm_Drill1.0mm, symbol Connector:TestPoint
- added TP?: Coupling, TestPoint:TestPoint_Pad_1.5x1.5mm, symbol Connector:TestPoint
- added U? (x9): TL072, AJ-Dropbox-Kicad:AJ_SO-8_5.3x6.2mm_P1.27mm, symbol Amplifier_Operational:TL072
Connections:
- net +12V: now also C?.1, C?.1, C?.1, D?.2 (A), P?.10 (+12), P?.9 (+12), Q?.3 (C), R?.1, R?.1, R?.2, R?.2, R?.2, R?.2, U?.4 (V-), U?.4 (V-), U?.4 (V-)
- net -12V: now also C?.2, C?.2, C?.2, D?.1 (K), P?.1 (-12), P?.2 (-12), U?.8 (V+), U?.8 (V+), U?.8 (V+)
- net Coupling: now also C?.2, Q?.3 (C), R?.2, R?.2, TP?.1
- net GND: now also C?.1, C?.1, C?.1, C?.2, C?.2, C?.2, C?.2, C?.2, C?.2, C?.2, D?.1 (K), D?.2 (A), D?.2 (A), D?.2 (A), D?.2 (A), D?.2 (A), J?.S, J?.S, J?.S, J?.TN, J?.TN, P?.3 (GND), P?.4 (GND), P?.5 (GND), P?.6 (GND), P?.7 (GND), P?.8 (GND), Q?.1 (B), Q?.2 (E), Q?.2 (E), Q?.2 (E), R?.1, R?.1, R?.1, R?.1, R?.1, R?.1, R?.1, R?.1, R?.1, R?.1, R?.2, R?.2, R?.2, R?.2, R?.2, R?.2, RV?.1, RV?.3, SW?.1 (A), TP?.1, U?.5 (+)
- net InAccent: now also D?.1 (K), R?.1, R?.1, R?.2, R?.2
- net InGate: now also C?.1, D?.1 (K), R?.1, R?.2, R?.2
- net NoiseIn: now also JP?.2, R?.2
- net OutTom: now also R?.2, R?.2
- net PNP_B: now also Q?.1 (B), R?.1, R?.2
- net PNP_E: now also Q?.2 (E), Q?.2 (E), R?.2, R?.2
- net PinkNoise: now also C?.1, RV?.3, U?.6 (-), U?.7
- net WhiteNoise: now also R?.1, R?.1, RV?.1, TP?.1, U?.1
- new net: C?.2, R?.1, R?.1, RV?.2, U?.1
- new net: C?.1, C?.2, R?.2, RV?.1, U?.2 (-)
- new net: R?.2, U?.3 (+)
- new net: R?.1, R?.2, U?.6 (-) (x2)
- new net: R?.1, R?.2, RV?.2, U?.7
- new net: R?.1, RV?.3
- new net: D?.1 (K), D?.2 (A), RV?.1
- new net: R?.1, RV?.2
- new net: C?.2, C?.2, R?.1, R?.1, U?.1
- new net: C?.1, R?.2, U?.2 (-)
- new net: R?.1, R?.1, R?.1, U?.3 (+)
- new net: R?.2, SW?.2 (B)
- new net: C?.1, SW?.5 (B)
- new net: C?.1, C?.2, D?.1 (K), D?.2 (A), R?.2, R?.2, SW?.6 (C)
- new net: R?.2, RV?.2 (x2)
- new net: C?.1, R?.2, RV?.3
- new net: R?.1, R?.2, U?.5 (+)
- new net: R?.1, R?.2, U?.7
- new net: Q?.1 (B), R?.1, R?.2 (x2)
- new net: Q?.3 (C), R?.1 (x2)
- new net: Q?.3 (C), R?.1, R?.2
- new net: C?.2, D?.1 (K), R?.2
- new net: Q?.1 (B), R?.1, R?.1
- new net: Q?.1 (B), R?.2 (x2)
- new net: Q?.2 (E), R?.1, R?.2
- new net: D?.2 (A), R?.1
- new net: C?.1, D?.1 (K), R?.1
- new net: C?.2, R?.1, R?.2 (x2)
- new net: C?.2, Q?.3 (C), R?.1
- new net: C?.1, R?.1, R?.2 (x3)
- new net: C?.1, D?.1 (K), R?.2
- new net: J?.T, R?.1 (x3)
- new net: R?.2, U?.2 (-)
- new net: C?.1, R?.1, U?.3 (+)
- new net: C?.1, R?.2, U?.5 (+)
- new net: C?.1, R?.2, R?.2
- new net: C?.2, Q?.2 (E), R?.1
- new net: R?.1, R?.2, RV?.1
- new net: JP?.1, RV?.2

Commit message: Main components placed
Parts:
- gave numbers to parts that had none: 113
Connections:
- net GND: now also SW201.4 (A); no longer SW201.1 (A)
- net at R230.2: now also SW201.5 (B); no longer SW201.2 (B)
- net at C211.1: now also SW201.2 (B); no longer SW201.5 (B)
- net at C212.2, C213.1, D205.2 (A)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: now also SW201.3 (C); no longer SW201.6 (C)
