File: KicadJE_AteOhAte - RevB/KicadJE_AteOhAte.kicad_pcb (KiCad board)
At the start: 2 copper layers, 100 x 100 mm, 202 parts, among them J201 In_Accent, J202 In Gate, J203 Out Tom, J301 PJRAS2X2S01AUX, J302 Conn_01x03, P201 Doepfer_Power_10pin, Q201 MMBT2222A, Q202 MMBT2222A, Q203 MMBT2222A, Q204 MMBT2222A, Q205 MMBT2907A, Q206 MMBT2222A, Q207 MMBT2222A, SW201 Con/Tom, U201 TL072, U202 TL072, U203 TL072, U301 TL072, U302 TL072, U303 TL072

Commit message: 2nd tom
Parts:
- removed C318, C322: 47p, Capacitor_SMD:C_0805_2012Metric_Pad1.15x1.40mm_HandSolder
- removed C319: 2n2, Capacitor_SMD:C_0805_2012Metric_Pad1.15x1.40mm_HandSolder
- removed C320: 1n_THT, Capacitor_THT:C_Rect_L7.2mm_W5.5mm_P5.00mm_FKS2_FKP2_MKS2_MKP2
- removed C321: 680p_THT, Capacitor_THT:C_Rect_L7.2mm_W5.5mm_P5.00mm_FKS2_FKP2_MKS2_MKP2
- removed C323: 1n, Capacitor_SMD:C_0805_2012Metric_Pad1.15x1.40mm_HandSolder
- removed C324: 680p, Capacitor_SMD:C_0805_2012Metric_Pad1.15x1.40mm_HandSolder
- removed C325, C329, C330: 470n_THT, Capacitor_THT:C_Rect_L7.2mm_W5.5mm_P5.00mm_FKS2_FKP2_MKS2_MKP2
- removed C326: 470n, Capacitor_SMD:C_1206_3216Metric_Pad1.42x1.75mm_HandSolder
- removed C327, C328: 470n, Capacitor_SMD:C_0805_2012Metric_Pad1.15x1.40mm_HandSolder
- removed C331, C343: 10u, Capacitor_THT:CP_Radial_D8.0mm_P3.50mm
- removed C332, C344: 22u, Capacitor_THT:CP_Radial_D8.0mm_P3.50mm
- removed C333, C341: 10u, Capacitor_SMD:C_0805_2012Metric_Pad1.15x1.40mm_HandSolder
- removed C334, C342: 1u, Capacitor_SMD:C_0805_2012Metric_Pad1.15x1.40mm_HandSolder
- removed C335, C336, C337, C338, C339, C340: 100n, Capacitor_SMD:C_0805_2012Metric_Pad1.15x1.40mm_HandSolder
- removed C345, C346: 470u, Capacitor_THT:CP_Radial_D13.0mm_P5.00mm
- removed F301, F302: Polyfuse, Fuse:Fuse_1206_3216Metric
- removed the G*** at (130.5, 64.5)
- removed the G*** at (121.5, 125.5)
- added C201: 10u, Capacitor_SMD:C_1206_3216Metric_Pad1.42x1.75mm_HandSolder, F.Cu at (-16.8, 7.80)
- added C202: 100n, Capacitor_SMD:C_0805_2012Metric_Pad1.15x1.40mm_HandSolder, F.Cu at (25.3, -1.84)
- added C203: 100n, Capacitor_SMD:C_0805_2012Metric_Pad1.15x1.40mm_HandSolder, F.Cu at (58.6, -34.2)
- added C204: 10u, Capacitor_SMD:C_1206_3216Metric_Pad1.42x1.75mm_HandSolder, F.Cu at (4.68, 6.36)
- added C205: 100n, Capacitor_SMD:C_0805_2012Metric_Pad1.15x1.40mm_HandSolder, F.Cu at (35.2, -13.8)
- added C206: 100n, Capacitor_SMD:C_0805_2012Metric_Pad1.15x1.40mm_HandSolder, F.Cu at (46.1, -24.7)
- added C207: 39n, Capacitor_SMD:C_0805_2012Metric_Pad1.15x1.40mm_HandSolder, F.Cu at (60.4, -38.7)
- added C208: 1u, Capacitor_SMD:C_0805_2012Metric_Pad1.15x1.40mm_HandSolder, F.Cu at (21.2, 1.39)
- added C209: 22u, Capacitor_SMD:C_0805_2012Metric_Pad1.15x1.40mm_HandSolder, F.Cu at (14.8, 7.59)
- added C210: 18n, Capacitor_SMD:C_0805_2012Metric_Pad1.15x1.40mm_HandSolder, F.Cu at (28.0, -5.19)
- added C211: C11, Capacitor_SMD:C_0805_2012Metric_Pad1.15x1.40mm_HandSolder, F.Cu at (51.3, -30.6)
- added C212: C9, Capacitor_SMD:C_0805_2012Metric_Pad1.15x1.40mm_HandSolder, F.Cu at (41.4, -19.8)
- added C213: C10, Capacitor_SMD:C_0805_2012Metric_Pad1.15x1.40mm_HandSolder, F.Cu at (-11.5, 7.63)
- added C214: 1n, Capacitor_SMD:C_0805_2012Metric_Pad1.15x1.40mm_HandSolder, F.Cu at (16.5, 4.34)
- added C215: C12, Capacitor_SMD:C_0805_2012Metric_Pad1.15x1.40mm_HandSolder, F.Cu at (34.8, -4.99)
- added C216: C8, Capacitor_SMD:C_0805_2012Metric_Pad1.15x1.40mm_HandSolder, F.Cu at (10.0, 7.59)
- added C217: C6, Capacitor_SMD:C_0805_2012Metric_Pad1.15x1.40mm_HandSolder, F.Cu at (16.5, 1.39)
- added C218: 47n, Capacitor_SMD:C_0805_2012Metric_Pad1.15x1.40mm_HandSolder, F.Cu at (35.2, -16.8)
- added C219: 10n, Capacitor_SMD:C_0805_2012Metric_Pad1.15x1.40mm_HandSolder, F.Cu at (41.4, -22.8)
- added C220: C7, Capacitor_SMD:C_0805_2012Metric_Pad1.15x1.40mm_HandSolder, F.Cu at (61.1, -41.7)
- added C221: C4, Capacitor_SMD:C_0805_2012Metric_Pad1.15x1.40mm_HandSolder, F.Cu at (35.5, -2.04)
- added D201: 1N1007, Diode_SMD:D_SOD-123, F.Cu at (30.0, -14.6)
- added D202: 1N1007, Diode_SMD:D_SOD-123, F.Cu at (61.6, -44.8)
- added D203: D_Zener, Diode_SMD:D_MiniMELF, F.Cu at (-29.3, 7.78)
- added D204: D_Zener, Diode_SMD:D_MiniMELF, F.Cu at (-23.0, 7.78)
- added D205: 1N4148, Diode_SMD:D_SOD-123, F.Cu at (55.1, -40.3)
- added D206: 1N4148, Diode_SMD:D_SOD-123, F.Cu at (48.6, -33.7)
- added D207: 1N4148, Diode_SMD:D_SOD-123, F.Cu at (40.6, -25.9)
- added D208: 1N4148, Diode_SMD:D_SOD-123, F.Cu at (30.0, -18.0)
- added D209: 1N4148, Diode_SMD:D_SOD-123, F.Cu at (22.7, -4.99)
- added D301: 1N1007, Diode_SMD:D_SOD-123, B.Cu at (285.6, 149.8)
- added D302: 1N1007, Diode_SMD:D_SOD-123, B.Cu at (216.0, 117.1)
- added D303: Zener, Diode_SMD:D_MiniMELF, B.Cu at (161.7, 133.2)
- added D305: Zener, Diode_SMD:D_MiniMELF, B.Cu at (256.0, 129.0)
- added D306: Zener, Diode_SMD:D_MiniMELF, B.Cu at (279.6, 149.9)
- added D307: Zener, Diode_SMD:D_MiniMELF, B.Cu at (174.4, 133.2)
- added D308: Zener, Diode_SMD:D_MiniMELF, B.Cu at (168.0, 133.2)
- added D309: 1N4148, Diode_SMD:D_SOD-123, B.Cu at (203.1, 104.9)
- added D310: 1N4148, Diode_SMD:D_SOD-123, B.Cu at (271.3, 137.5)
- added D311: 1N4148, Diode_SMD:D_SOD-123, B.Cu at (262.0, 128.9)
- added D312: 1N4148, Diode_SMD:D_SOD-123, B.Cu at (279.3, 146.6)
- added D313: 1N4148, Diode_SMD:D_SOD-123, B.Cu at (275.0, 142.1)
- added H203: 2,2mm, MountingHole:MountingHole_2.2mm_M2_Pad_Via, F.Cu at (36.0, -21.2)
- added H204: 2,2mm, MountingHole:MountingHole_2.2mm_M2_Pad_Via, F.Cu at (11.1, 3.14)
- added H302: 2,5mm, MountingHole:MountingHole_2.5mm_Pad_Via, B.Cu at (197.0, 112.4)
- added H304: 2,2mm, MountingHole:MountingHole_2.2mm_M2_Pad_Via, B.Cu at (255.8, 124.4)
- added J201: In_Accent, Connector_Audio:Jack_3.5mm_Ledino_KB3SPRS_Horizontal, F.Cu at (17.9, -78.6)
- added J202: In Gate, AJ-Dropbox-Kicad:PJ301SM, F.Cu at (-3.37, 0.29)
- added J203: Out Tom, AJ-Dropbox-Kicad:PJ301SM, F.Cu at (40.6, -39.9)
- added J303: In Gate, AJ-Dropbox-Kicad:PJ301SM, F.Cu at (223.0, 56.0)
- added J304: Out Tom, AJ-Dropbox-Kicad:PJ301SM, F.Cu at (237.6, 39.1)
- added JP201: Jumper, Connector_PinHeader_2.54mm:PinHeader_1x02_P2.54mm_Vertical, F.Cu at (18.2, -15.4)
- added P201: Doepfer_Power_10pin, Connectors_IDC:IDC-Header_2x05_Pitch2.54mm_Straight, F.Cu at (-11.0, -60.6)
- added P301: Doepfer_Power_10pin, Connectors_IDC:IDC-Header_2x05_Pitch2.54mm_Straight, F.Cu at (105.0, 56.0)
- added Q201: MMBT2222A, Package_TO_SOT_SMD:SOT-23_Handsoldering, F.Cu at (29.8, -21.9)
- added Q202: MMBT2222A, Package_TO_SOT_SMD:SOT-23_Handsoldering, F.Cu at (4.93, 2.44)
- added Q203: MMBT2222A, Package_TO_SOT_SMD:SOT-23_Handsoldering, F.Cu at (16.6, -5.31)
- added Q204: MMBT2222A, Package_TO_SOT_SMD:SOT-23_Handsoldering, F.Cu at (23.8, -8.94)
- added Q205: MMBT2907A, Package_TO_SOT_SMD:SOT-23_Handsoldering, F.Cu at (55.5, -44.2)
- added Q206: MMBT2222A, Package_TO_SOT_SMD:SOT-23_Handsoldering, F.Cu at (48.9, -37.7)
- added Q207: MMBT2222A, Package_TO_SOT_SMD:SOT-23_Handsoldering, F.Cu at (41.0, -29.9)
- added Q301: MMBT2222A, Package_TO_SOT_SMD:SOT-23_Handsoldering, B.Cu at (203.5, 113.4)
- added Q302: MMBT2222A, Package_TO_SOT_SMD:SOT-23_Handsoldering, B.Cu at (268.9, 141.5)
- added Q303: MMBT2222A, Package_TO_SOT_SMD:SOT-23_Handsoldering, B.Cu at (203.5, 108.8)
- added Q304: MMBT2907A, Package_TO_SOT_SMD:SOT-23_Handsoldering, B.Cu at (197.0, 102.3)
- added Q305: MMBT2222A, Package_TO_SOT_SMD:SOT-23_Handsoldering, B.Cu at (216.4, 124.3)
- added Q306: MMBT2222A, Package_TO_SOT_SMD:SOT-23_Handsoldering, B.Cu at (197.0, 106.8)
- added R201: 1M, Resistor_SMD:R_0805_2012Metric_Pad1.15x1.40mm_HandSolder, F.Cu at (54.5, -37.1)
- added R202: 4k7, Resistor_SMD:R_0805_2012Metric_Pad1.15x1.40mm_HandSolder, F.Cu at (46.6, -30.6)
- added R203: 330K, Resistor_SMD:R_0805_2012Metric_Pad1.15x1.40mm_HandSolder, F.Cu at (29.4, -9.74)
- added R204: 100R, Resistor_SMD:R_0805_2012Metric_Pad1.15x1.40mm_HandSolder, F.Cu at (46.6, -27.6)
- added R205: 22k, Resistor_SMD:R_0805_2012Metric_Pad1.15x1.40mm_HandSolder, F.Cu at (20.5, -1.56)
- added R206: 1M, Resistor_SMD:R_0805_2012Metric_Pad1.15x1.40mm_HandSolder, F.Cu at (53.8, -33.9)
- added R207: 22k, Resistor_SMD:R_0805_2012Metric_Pad1.15x1.40mm_HandSolder, F.Cu at (34.1, -10.9)
- added R208: 300R, Resistor_SMD:R_0805_2012Metric_Pad1.15x1.40mm_HandSolder, F.Cu at (51.3, -27.6)
- added R209: 1K, Resistor_SMD:R_0805_2012Metric_Pad1.15x1.40mm_HandSolder, F.Cu at (40.0, -16.8)
- added R210: OPEN, Resistor_SMD:R_0805_2012Metric_Pad1.15x1.40mm_HandSolder, F.Cu at (65.8, -41.7)
- added R211: 1K, Resistor_SMD:R_0805_2012Metric_Pad1.15x1.40mm_HandSolder, F.Cu at (60.4, -22.4)
- added R212: 0R, Resistor_SMD:R_0805_2012Metric_Pad1.15x1.40mm_HandSolder, F.Cu at (48.4, -9.92)
- added R213: OPEN, Resistor_SMD:R_0805_2012Metric_Pad1.15x1.40mm_HandSolder, F.Cu at (54.2, -15.8)
- added R214: 1k, Resistor_SMD:R_0805_2012Metric_Pad1.15x1.40mm_HandSolder, F.Cu at (65.6, -26.9)
- added R215: 470k, Resistor_SMD:R_0805_2012Metric_Pad1.15x1.40mm_HandSolder, F.Cu at (44.3, -6.97)
- added R216: 820k, Resistor_SMD:R_0805_2012Metric_Pad1.15x1.40mm_HandSolder, F.Cu at (30.0, -2.24)
- added R217: 33k, Resistor_SMD:R_0805_2012Metric_Pad1.15x1.40mm_HandSolder, F.Cu at (21.2, 4.34)
- added R218: 100k, Resistor_SMD:R_0805_2012Metric_Pad1.15x1.40mm_HandSolder, F.Cu at (56.1, -31.0)
- added R219: 100k, Resistor_SMD:R_0805_2012Metric_Pad1.15x1.40mm_HandSolder, F.Cu at (40.0, -13.8)
- added R220: 4k7, Resistor_SMD:R_0805_2012Metric_Pad1.15x1.40mm_HandSolder, F.Cu at (34.1, -7.94)
- added R221: 4k7, Resistor_SMD:R_0805_2012Metric_Pad1.15x1.40mm_HandSolder, F.Cu at (50.9, -24.7)
- added R222: 470k, Resistor_SMD:R_0805_2012Metric_Pad1.15x1.40mm_HandSolder, F.Cu at (46.1, -18.8)
- added R223: 33k, Resistor_SMD:R_0805_2012Metric_Pad1.15x1.40mm_HandSolder, F.Cu at (65.1, -38.7)
- added R224: 100k, Resistor_SMD:R_0805_2012Metric_Pad1.15x1.40mm_HandSolder, F.Cu at (26.0, 1.11)
- added R225: 1k, Resistor_SMD:R_0805_2012Metric_Pad1.15x1.40mm_HandSolder, F.Cu at (55.6, -21.7)
- added R226: 15k, Resistor_SMD:R_0805_2012Metric_Pad1.15x1.40mm_HandSolder, F.Cu at (38.9, -10.9)
- added R227: 10k, Resistor_SMD:R_0805_2012Metric_Pad1.15x1.40mm_HandSolder, F.Cu at (56.1, -28.0)
- added R228: 4k7, Resistor_SMD:R_0805_2012Metric_Pad1.15x1.40mm_HandSolder, F.Cu at (46.1, -21.7)
- added R229: 4k7, Resistor_SMD:R_0805_2012Metric_Pad1.15x1.40mm_HandSolder, F.Cu at (63.3, -35.8)
- added R230: R17, Resistor_SMD:R_0805_2012Metric_Pad1.15x1.40mm_HandSolder, F.Cu at (50.9, -21.7)
- added R231: R18, Resistor_SMD:R_0805_2012Metric_Pad1.15x1.40mm_HandSolder, F.Cu at (26.0, 4.06)
- added R232: 22k, Resistor_SMD:R_0805_2012Metric_Pad1.15x1.40mm_HandSolder, F.Cu at (60.8, -31.2)
- added R233: 4k7, Resistor_SMD:R_0805_2012Metric_Pad1.15x1.40mm_HandSolder, F.Cu at (44.7, -15.8)
- added R234: 100k, Resistor_SMD:R_0805_2012Metric_Pad1.15x1.40mm_HandSolder, F.Cu at (38.9, -7.94)
- added R235: 4k7, Resistor_SMD:R_0805_2012Metric_Pad1.15x1.40mm_HandSolder, F.Cu at (55.6, -24.7)
- added R236: 10k, Resistor_SMD:R_0805_2012Metric_Pad1.15x1.40mm_HandSolder, F.Cu at (50.9, -18.8)
- added R237: 10k, Resistor_SMD:R_0805_2012Metric_Pad1.15x1.40mm_HandSolder, F.Cu at (44.7, -12.9)
- added R238: 4k7, Resistor_SMD:R_0805_2012Metric_Pad1.15x1.40mm_HandSolder, F.Cu at (24.3, 7.29)
- added R239: 4k7, Resistor_SMD:R_0805_2012Metric_Pad1.15x1.40mm_HandSolder, F.Cu at (30.7, 0.71)
- added R240: 22k, Resistor_SMD:R_0805_2012Metric_Pad1.15x1.40mm_HandSolder, F.Cu at (19.5, 7.29)
- added R241: 22k, Resistor_SMD:R_0805_2012Metric_Pad1.15x1.40mm_HandSolder, F.Cu at (15.8, -1.56)
- added R242: 4k7, Resistor_SMD:R_0805_2012Metric_Pad1.15x1.40mm_HandSolder, F.Cu at (49.5, -15.8)
- added R243: 3k3, Resistor_SMD:R_0805_2012Metric_Pad1.15x1.40mm_HandSolder, F.Cu at (30.7, 3.66)
- added R244: 33k, Resistor_SMD:R_0805_2012Metric_Pad1.15x1.40mm_HandSolder, F.Cu at (39.5, -4.99)
- added R245: 22k, Resistor_SMD:R_0805_2012Metric_Pad1.15x1.40mm_HandSolder, F.Cu at (65.6, -32.8)
- added R246: 10k, Resistor_SMD:R_0805_2012Metric_Pad1.15x1.40mm_HandSolder, F.Cu at (43.6, -9.92)
- added R247: 47k, Resistor_SMD:R_0805_2012Metric_Pad1.15x1.40mm_HandSolder, F.Cu at (60.8, -25.3)
- added R248: 2M2, Resistor_SMD:R_0805_2012Metric_Pad1.15x1.40mm_HandSolder, F.Cu at (55.6, -18.8)
- added R249: 33k, Resistor_SMD:R_0805_2012Metric_Pad1.15x1.40mm_HandSolder, F.Cu at (65.6, -29.9)
- added R250: 22k, Resistor_SMD:R_0805_2012Metric_Pad1.15x1.40mm_HandSolder, F.Cu at (49.5, -12.9)
- added R251: 100k, Resistor_SMD:R_0805_2012Metric_Pad1.15x1.40mm_HandSolder, F.Cu at (60.8, -28.3)
- added R252: 100k, Resistor_SMD:R_0805_2012Metric_Pad1.15x1.40mm_HandSolder, F.Cu at (35.5, 0.91)
- added R253: 100k, Resistor_SMD:R_0805_2012Metric_Pad1.15x1.40mm_HandSolder, F.Cu at (29.0, 7.01)
- added R254: 100k, Resistor_SMD:R_0805_2012Metric_Pad1.15x1.40mm_HandSolder, F.Cu at (40.2, -2.04)
- added R331: 10k, Resistor_SMD:R_0805_2012Metric_Pad1.15x1.40mm_HandSolder, B.Cu at (267.2, 119.9)
- added R332: 4k7, Resistor_SMD:R_0805_2012Metric_Pad1.15x1.40mm_HandSolder, B.Cu at (276.8, 130.1)
- added R333: 4k7, Resistor_SMD:R_0805_2012Metric_Pad1.15x1.40mm_HandSolder, B.Cu at (257.0, 113.6)
- added R334: 22k, Resistor_SMD:R_0805_2012Metric_Pad1.15x1.40mm_HandSolder, B.Cu at (261.8, 114.0)
- added R335: 22k, Resistor_SMD:R_0805_2012Metric_Pad1.15x1.40mm_HandSolder, B.Cu at (286.1, 137.8)
- added R336: 4k7, Resistor_SMD:R_0805_2012Metric_Pad1.15x1.40mm_HandSolder, B.Cu at (255.6, 107.4)
- added R337: 3k3, Resistor_SMD:R_0805_2012Metric_Pad1.15x1.40mm_HandSolder, B.Cu at (272.0, 123.2)
- added R338: 33k, Resistor_SMD:R_0805_2012Metric_Pad1.15x1.40mm_HandSolder, B.Cu at (216.8, 102.2)
- added R339: 22k, Resistor_SMD:R_0805_2012Metric_Pad1.15x1.40mm_HandSolder, B.Cu at (276.8, 127.1)
- added R340: 10k, Resistor_SMD:R_0805_2012Metric_Pad1.15x1.40mm_HandSolder, B.Cu at (260.3, 110.7)
- added R341: 47k, Resistor_SMD:R_0805_2012Metric_Pad1.15x1.40mm_HandSolder, B.Cu at (266.7, 116.9)
- added R342: 2M2, Resistor_SMD:R_0805_2012Metric_Pad1.15x1.40mm_HandSolder, B.Cu at (254.4, 104.1)
- added R343: 33k, Resistor_SMD:R_0805_2012Metric_Pad1.15x1.40mm_HandSolder, B.Cu at (284.7, 134.6)
- added R344: 22k, Resistor_SMD:R_0805_2012Metric_Pad1.15x1.40mm_HandSolder, B.Cu at (217.8, 105.1)
- added R345: 100k, Resistor_SMD:R_0805_2012Metric_Pad1.15x1.40mm_HandSolder, B.Cu at (276.7, 124.2)
- added R346: 100k, Resistor_SMD:R_0805_2012Metric_Pad1.15x1.40mm_HandSolder, B.Cu at (253.6, 101.1)
- added R347: 100k, Resistor_SMD:R_0805_2012Metric_Pad1.15x1.40mm_HandSolder, B.Cu at (266.5, 114.0)
- added R348: 100k, Resistor_SMD:R_0805_2012Metric_Pad1.15x1.40mm_HandSolder, B.Cu at (260.3, 107.7)
- added RV201: 100K, Potentiometer_THT:Potentiometer_Bourns_3296W_Vertical, F.Cu at (22.0, -66.0)
- added RV202: 50K, Potentiometer_THT:Potentiometer_Bourns_3296W_Vertical, F.Cu at (3.84, -48.8)
- added RV203: 500R Tune, Potentiometer_THT:Potentiometer_Piher_T-16H_Single_Horizontal, F.Cu at (-38.7, -77.7)
- added RV204: 1M Decay, Potentiometer_THT:Potentiometer_Piher_T-16H_Single_Horizontal, F.Cu at (-9.67, -76.7)
- added RV205: 100k A Level, Potentiometer_THT:Potentiometer_Piher_T-16H_Single_Horizontal, F.Cu at (-38.7, -42.6)
- added RV206: 100k A Reverb, Potentiometer_THT:Potentiometer_Piher_T-16H_Single_Horizontal, F.Cu at (-38.7, -60.2)
- added RV301: 500R Tune, Potentiometer_THT:Potentiometer_Piher_T-16H_Single_Horizontal, F.Cu at (148.0, 64.0)
- added RV302: 1M Decay, Potentiometer_THT:Potentiometer_Piher_T-16H_Single_Horizontal, F.Cu at (148.0, 104.0)
- added RV303: 100k A Level, Potentiometer_THT:Potentiometer_Piher_T-16H_Single_Horizontal, F.Cu at (148.0, 125.0)
- added RV304: 100k A Reverb, Potentiometer_THT:Potentiometer_Piher_T-16H_Single_Horizontal, F.Cu at (148.0, 84.0)
- added SW201: Con/Tom, AJ-Dropbox-Kicad:SPDTx2, F.Cu at (2.31, -59.5)
- added SW301: Con/Tom, AJ-Dropbox-Kicad:SPDTx2, F.Cu at (252.0, 39.0)
- added TP201: WhiteNoise, TestPoint:TestPoint_Pad_1.5x1.5mm, F.Cu at (59.8, -19.1)
- added TP202: GND, TestPoint:TestPoint_THTPad_2.0x2.0mm_Drill1.0mm, F.Cu at (35.1, 4.41)
- added TP203: Coupling, TestPoint:TestPoint_Pad_1.5x1.5mm, F.Cu at (53.6, -12.6)
- added TP301: Coupling, TestPoint:TestPoint_Pad_1.5x1.5mm, B.Cu at (270.9, 116.6)
- added U201: TL072, AJ-Dropbox-Kicad:AJ_SO-8_5.3x6.2mm_P1.27mm, F.Cu at (21.3, -21.6)
- added U202: TL072, AJ-Dropbox-Kicad:AJ_SO-8_5.3x6.2mm_P1.27mm, F.Cu at (8.07, -3.71)
- added U203: TL072, AJ-Dropbox-Kicad:AJ_SO-8_5.3x6.2mm_P1.27mm, F.Cu at (32.4, -28.1)
- C301: value 2n2_THT -> 10u; footprint Capacitor_THT:C_Rect_L7.2mm_W5.5mm_P5.00mm_FKS2_FKP2_MKS2_MKP2 -> Capacitor_SMD:C_1206_3216Metric_Pad1.42x1.75mm_HandSolder; moved to B.Cu
- C302: value 100u -> 100n; footprint Capacitor_SMD:CP_Elec_8x6.5 -> Capacitor_SMD:C_0805_2012Metric_Pad1.15x1.40mm_HandSolder; moved to B.Cu
- C303: value 2n2 -> 100n
- C304: value 1n_THT -> 10u; footprint Capacitor_THT:C_Rect_L7.2mm_W5.5mm_P5.00mm_FKS2_FKP2_MKS2_MKP2 -> Capacitor_SMD:C_1206_3216Metric_Pad1.42x1.75mm_HandSolder; moved to B.Cu
- C305: value 680p_THT -> 100n; footprint Capacitor_THT:C_Rect_L7.2mm_W5.5mm_P5.00mm_FKS2_FKP2_MKS2_MKP2 -> Capacitor_SMD:C_0805_2012Metric_Pad1.15x1.40mm_HandSolder; moved to B.Cu
- C306: value 47p -> 100n
- C307: value 1n -> C11
- C308: value 680p -> C9
- C309: value 470n_THT -> C10; footprint Capacitor_THT:C_Rect_L7.2mm_W5.5mm_P5.00mm_FKS2_FKP2_MKS2_MKP2 -> Capacitor_SMD:C_0805_2012Metric_Pad1.15x1.40mm_HandSolder; moved to B.Cu
- C310: value 47p -> 1n
- C311: value 470n -> C12; footprint Capacitor_SMD:C_1206_3216Metric_Pad1.42x1.75mm_HandSolder -> Capacitor_SMD:C_0805_2012Metric_Pad1.15x1.40mm_HandSolder
- C312: value 470n -> C8
- C313: value 470n -> C6
- C314: value 470n_THT -> 47n; footprint Capacitor_THT:C_Rect_L7.2mm_W5.5mm_P5.00mm_FKS2_FKP2_MKS2_MKP2 -> Capacitor_SMD:C_0805_2012Metric_Pad1.15x1.40mm_HandSolder; moved to B.Cu
- C315: value 470n_THT -> 10n; footprint Capacitor_THT:C_Rect_L7.2mm_W5.5mm_P5.00mm_FKS2_FKP2_MKS2_MKP2 -> Capacitor_SMD:C_0805_2012Metric_Pad1.15x1.40mm_HandSolder; moved to B.Cu
- C316: value 100u -> C7; footprint Capacitor_SMD:CP_Elec_8x6.5 -> Capacitor_SMD:C_0805_2012Metric_Pad1.15x1.40mm_HandSolder; moved to B.Cu
- C317: value 2n2_THT -> C4; footprint Capacitor_THT:C_Rect_L7.2mm_W5.5mm_P5.00mm_FKS2_FKP2_MKS2_MKP2 -> Capacitor_SMD:C_0805_2012Metric_Pad1.15x1.40mm_HandSolder; moved to B.Cu
- D304: value LED -> Zener; footprint LED_THT:LED_D3.0mm -> Diode_SMD:D_MiniMELF; moved to B.Cu
- H301: moved to B.Cu
- H303: value 2,5mm -> 2,2mm; footprint MountingHole:MountingHole_2.5mm_Pad_Via -> MountingHole:MountingHole_2.2mm_M2_Pad_Via; moved to B.Cu
- J301: value PJRAS2X2S01AUX -> Noise_In; footprint AJ:PJRAS2X2S01AUX_RCA -> Connector_Audio:Jack_3.5mm_Ledino_KB3SPRS_Horizontal
- J302: value Conn_01x03 -> In_Accent; footprint TerminalBlock:TerminalBlock_bornier-3_P5.08mm -> Connector_Audio:Jack_3.5mm_Ledino_KB3SPRS_Horizontal
- R301: value 220R -> 1K
- R302, R305: value 2k2 -> 1K
- R303: value 82k -> OPEN
- R304: value 2k2 -> OPEN
- R306: value 470R -> OPEN
- R307: value 470R -> 0R
- R308: value 18k -> 1k
- R309: value 1M -> 470k
- R310: value 47k -> 820k
- R311, R317: value 470R -> 33k
- R312, R313: value 18k -> 100k
- R314: value 220R -> 4k7
- R315: value 2k2 -> 4k7
- R316: value 82k -> 470k
- R318: value 470R -> 100k
- R319: value 2k2 -> 1k
- R320: value 2k2 -> 15k
- R321: value 47k -> 10k
- R322: value 18k -> 4k7
- R323: value 1M -> 4k7
- R324: value 470R -> R17
- R325: value 18k -> R18
- R326: value 680k -> 22k
- R327: value 12k -> 4k7
- R328: value 680k -> 100k
- R329: value 1R1 -> 4k7
- R330: value 1R1 -> 10k
- moved H201 194.5 mm to (23.8, -14.5)
- moved H202 192.6 mm to (49.0, -43.2)
- moved C307 178.2 mm to (280.3, 143.4), turned to 0 degrees
- moved R309 176.5 mm to (281.5, 127.1), turned to 0 degrees
- moved R303 172.8 mm to (276.6, 136.0), turned to 0 degrees
- moved R330 170.1 mm to (279.9, 133.0), turned to 0 degrees
- moved R312 168.1 mm to (275.2, 133.0)
- moved R311 161.8 mm to (267.2, 122.8)
- moved R302 161.0 mm to (284.5, 146.7), turned to 0 degrees
- moved R301 159.3 mm to (276.6, 138.9), turned to 0 degrees
- moved C304 159.2 mm to (265.1, 132.3), turned to 0 degrees
- moved U302 158.5 mm to (271.1, 147.6)
- moved C317 158.2 mm to (261.1, 125.8)
- moved R327 157.4 mm to (262.0, 116.9), turned to 0 degrees
- moved R320 157.3 mm to (281.5, 130.1)
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Connections:
- C301 pad 2: Net-(C301-Pad2) -> (no net)
- C302 pad 2: GND -> (no net)
- C303 pad 1: Net-(C301-Pad1) -> Net-(C303-Pad1)
- C303 pad 2: Net-(C301-Pad2) -> (no net)
- C304 pad 1: Net-(C301-Pad2) -> (no net)
- C304 pad 2: Net-(C304-Pad2) -> Net-(C301-Pad1)
- C305 pad 1: Net-(C301-Pad1) -> (no net)
- C305 pad 2: Net-(C301-Pad2) -> Net-(C302-Pad1)
- C306 pad 1: Net-(C306-Pad1) -> (no net)
- C306 pad 2: Net-(C306-Pad2) -> Net-(C303-Pad1)
- C307 pad 1: Net-(C301-Pad2) -> Net-(C307-Pad1)
- C307 pad 2: Net-(C304-Pad2) -> Net-(C307-Pad2)
- C308 pad 1: Net-(C301-Pad1) -> Net-(C308-Pad1)
- C308 pad 2: Net-(C301-Pad2) -> Net-(C308-Pad2)
- C309 pad 1: Net-(C309-Pad1) -> Net-(C308-Pad2)
- C309 pad 2: L_Rumble_Out -> Net-(C307-Pad2)
- C310 pad 2: GND -> Net-(C310-Pad2)
- C311 pad 1: Net-(C309-Pad1) -> Net-(C311-Pad1)
- C311 pad 2: L_Rumble_Out -> Net-(C310-Pad1)
- C312 pad 2: L_GainOut -> /KicadJE_AteOhAte3/Coupling
- C313 pad 2: Net-(C312-Pad1) -> Net-(C313-Pad2)
- C314 pad 1: Net-(C312-Pad1) -> Net-(C314-Pad1)
- C314 pad 2: L_GainOut -> Net-(C314-Pad2)
- C315 pad 1: Net-(C313-Pad1) -> InGate
- C315 pad 2: Net-(C312-Pad1) -> Net-(C315-Pad2)
- C317 pad 2: Net-(C317-Pad2) -> GND
- D304 pad 1: Net-(D304-Pad1) -> InAccent
- R301 pad 1: Net-(C306-Pad1) -> Net-(J301-PadT)
- R301 pad 2: Net-(C302-Pad1) -> NoiseIn
- R302 pad 1: L_GainOut -> Net-(J302-PadT)
- R302 pad 2: Net-(C306-Pad1) -> InAccent
- R303 pad 1: Net-(C301-Pad2) -> NoiseIn
- R303 pad 2: Net-(C304-Pad2) -> GND
- R304 pad 1: Net-(R304-Pad1) -> InAccent
- R305 pad 1: L_Rumble_Out -> Net-(J303-PadT)
- R305 pad 2: Net-(R304-Pad1) -> InGate
- R306 pad 1: Net-(C310-Pad1) -> InGate
- R306 pad 2: In_L -> GND
- R307 pad 1: Net-(C306-Pad2) -> Net-(J304-PadT)
- R307 pad 2: Net-(C310-Pad1) -> OutTom
- R308 pad 1: Net-(C304-Pad2) -> Net-(R308-Pad1)
- R308 pad 2: Net-(C309-Pad1) -> Net-(C308-Pad2)
- R309 pad 1: Net-(C301-Pad1) -> Net-(R309-Pad1)
- R309 pad 2: Net-(C304-Pad2) -> Net-(C308-Pad2)
- R310 pad 1: GND -> Net-(C307-Pad2)
- R310 pad 2: Net-(C310-Pad1) -> Net-(C308-Pad1)
- R311 pad 1: Out_L -> Net-(R311-Pad1)
- R311 pad 2: Net-(C301-Pad1) -> Net-(R311-Pad2)
- R312 pad 1: L_Rumble_Out -> InAccent
- R312 pad 2: Net-(C312-Pad1) -> +12V
- R313 pad 1: GND -> Net-(Q301-Pad1)
- R313 pad 2: Net-(C313-Pad1) -> +12V
- R314 pad 1: Net-(C318-Pad1) -> Net-(Q302-Pad3)
- R314 pad 2: Net-(C316-Pad1) -> InAccent
- R315 pad 1: R_GainOut -> Net-(Q301-Pad1)
- R315 pad 2: Net-(C318-Pad1) -> Net-(Q302-Pad3)
- R316 pad 1: Net-(C317-Pad2) -> Net-(C310-Pad2)
- R316 pad 2: Net-(C320-Pad2) -> Net-(C310-Pad1)
- R317 pad 1: Net-(C322-Pad1) -> Net-(C307-Pad2)
- R317 pad 2: In_R -> Net-(R311-Pad1)
- R318 pad 1: Net-(C318-Pad2) -> Net-(R311-Pad2)
- R318 pad 2: Net-(C322-Pad1) -> Net-(C311-Pad1)
- R319 pad 1: Net-(R319-Pad1) -> Net-(C310-Pad2)
- R319 pad 2: GND -> OutTom
- R320 pad 1: R_Rumble_Out -> Net-(Q303-Pad3)
- R320 pad 2: Net-(R319-Pad1) -> Net-(Q302-Pad1)
- R321 pad 1: GND -> Net-(Q302-Pad2)
- R321 pad 2: Net-(C322-Pad1) -> +12V
- R322 pad 1: Net-(C320-Pad2) -> GND
- R322 pad 2: Net-(C325-Pad1) -> /KicadJE_AteOhAte3/PNP_E
- R323 pad 1: Net-(C317-Pad1) -> /KicadJE_AteOhAte3/PNP_B
- R323 pad 2: Net-(C320-Pad2) -> /KicadJE_AteOhAte3/PNP_E
- R324 pad 1: Out_R -> Net-(R324-Pad1)
- R324 pad 2: Net-(C317-Pad1) -> Net-(R324-Pad2)
- R325 pad 1: R_Rumble_Out -> Net-(R324-Pad1)
- R325 pad 2: Net-(C327-Pad1) -> GND
- R326 pad 1: Net-(C331-Pad2) -> Net-(R324-Pad1)
- R326 pad 2: GND -> (no net)
- R327 pad 1: Net-(F301-Pad2) -> GND
- R327 pad 2: Net-(D304-Pad2) -> Net-(R327-Pad2)
- R328 pad 1: GND -> Net-(C311-Pad1)
- R328 pad 2: Net-(C341-Pad1) -> Net-(R328-Pad2)
- R329 pad 1: +12V -> GND
- R329 pad 2: Net-(F301-Pad2) -> Net-(Q302-Pad2)
- R330 pad 1: -12V -> Net-(Q305-Pad3)
- R330 pad 2: Net-(D304-Pad1) -> /KicadJE_AteOhAte3/PNP_B
- U301 pad 1: L_GainOut -> Net-(C307-Pad2)
- U301 pad 2: Net-(C306-Pad1) -> Net-(C308-Pad1)
- U301 pad 3: Net-(C306-Pad2) -> Net-(R324-Pad1)
- U301 pad 4: -12V -> /KicadJE_AteOhAte3/+12v
- U301 pad 5: Net-(C318-Pad2) -> GND
- U301 pad 6: Net-(C318-Pad1) -> Net-(R311-Pad1)
- U301 pad 7: R_GainOut -> Net-(R311-Pad2)
- U301 pad 8: +12V -> /KicadJE_AteOhAte3/-12v
- U302 pad 1: L_Rumble_Out -> Net-(C310-Pad2)
- U302 pad 2: Net-(R304-Pad1) -> Net-(C310-Pad1)
- U302 pad 3: Net-(C313-Pad1) -> Net-(R327-Pad2)
- U302 pad 4: -12V -> (no net)
- U302 pad 6: Net-(R319-Pad1) -> Net-(R347-Pad2)
- U302 pad 7: R_Rumble_Out -> Net-(R334-Pad1)
- U302 pad 8: +12V -> (no net)
- U303 pad 1: Net-(C301-Pad1) -> (no net)
- U303 pad 2: Net-(C304-Pad2) -> (no net)
- U303 pad 3: GND -> (no net)
- U303 pad 4: -12V -> (no net)
- U303 pad 5: GND -> (no net)
- U303 pad 6: Net-(C320-Pad2) -> (no net)
- U303 pad 7: Net-(C317-Pad1) -> (no net)
- U303 pad 8: +12V -> (no net)
Routing:
- net +12V: track 359.5 -> 238.2 mm
- net Net-(D304-Pad1): track 86.5 -> 0.00 mm
- net -12V: track 225.6 -> 157.3 mm, vias 2 -> 0
- net Net-(C310-Pad1): track 62.1 -> 0.00 mm, vias 2 -> 0
- net Out_L: track 56.0 -> 0.00 mm
- net Net-(C325-Pad1): track 49.0 -> 0.00 mm
- net Net-(C317-Pad1): track 42.8 -> 0.00 mm
- net Net-(C304-Pad2): track 32.6 -> 0.00 mm
- net Net-(D304-Pad2): track 32.0 -> 0.00 mm
- net Net-(C322-Pad1): track 30.5 -> 0.00 mm
- net Net-(C301-Pad1): track 28.4 -> 0.00 mm
- net Net-(C306-Pad1): track 25.4 -> 0.00 mm, vias 2 -> 0
- net Net-(C312-Pad1): track 23.6 -> 0.00 mm, vias 2 -> 0
- net L_Rumble_Out: track 21.3 -> 0.00 mm
- net Net-(C320-Pad2): track 21.0 -> 0.00 mm
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Other:
- board text removed: "+12V"
- board text removed: "-12V"
- board text removed: "Input"
- board text removed: "Input Gain Stage"
- board text removed: "Output"
- board text removed: "RIAA"
- board text removed: "RIAA Johansen Engineering Rev A - 27/09-2019"
- board text removed: "Rumble filter"

Commit message: Main components placed
Parts:
- removed U303: TL072, AJ-Dropbox-Kicad:AJ_SO-8_5.3x6.2mm_P1.27mm
- J301: footprint Connector_Audio:Jack_3.5mm_Ledino_KB3SPRS_Horizontal -> AJ-Dropbox-Kicad:PJ301SM
- moved D301 207.4 mm to (107.0, 44.5)
- moved C304 179.4 mm to (102.0, 57.5), turned to 270 degrees
- moved SW301 166.1 mm to (107.0, 120.0), turned to 180 degrees
- moved J304 161.4 mm to (115.0, 144.0), turned to 180 degrees
- moved U302 155.4 mm to (120.0, 111.0)
- moved J301 153.6 mm to (106.0, 144.0), turned to 180 degrees
- moved C302 148.4 mm to (123.0, 115.5)
- moved C305 143.5 mm to (117.0, 65.5)
- moved C303 140.8 mm to (123.0, 74.5)
- moved H301 140.4 mm to (140.0, 59.0)
- moved D306 139.6 mm to (140.1, 155.9)
- moved D304 139.2 mm to (128.2, 160.0)
- moved J303 131.7 mm to (125.0, 144.0), turned to 180 degrees
- moved D305 130.2 mm to (128.5, 155.5)
- moved C301 127.1 mm to (102.0, 64.5), turned to 270 degrees
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Connections:
- C301 pad 1: Net-(C301-Pad1) -> GND
- C301 pad 2: (no net) -> -12V
- C302 pad 1: Net-(C302-Pad1) -> GND
- C302 pad 2: (no net) -> -12V
- C303 pad 1: Net-(C303-Pad1) -> GND
- C303 pad 2: (no net) -> -12V
- C304 pad 1: (no net) -> +12V
- C304 pad 2: Net-(C301-Pad1) -> GND
- C305 pad 1: (no net) -> +12V
- C305 pad 2: Net-(C302-Pad1) -> GND
- C306 pad 1: (no net) -> +12V
- C306 pad 2: Net-(C303-Pad1) -> GND
- D301 pad 1: (no net) -> -12V
- D301 pad 2: Net-(D301-Pad2) -> GND
- D302 pad 1: Net-(D301-Pad2) -> GND
- D302 pad 2: (no net) -> +12V
- P301 pad 1: /KicadJE_AteOhAte3/-12v -> -12V
- P301 pad 10: /KicadJE_AteOhAte3/+12v -> +12V
- P301 pad 2: /KicadJE_AteOhAte3/-12v -> -12V
- P301 pad 9: /KicadJE_AteOhAte3/+12v -> +12V
- U301 pad 4: /KicadJE_AteOhAte3/+12v -> +12V
- U301 pad 8: /KicadJE_AteOhAte3/-12v -> -12V
- U302 pad 4: (no net) -> +12V
- U302 pad 8: (no net) -> -12V

Commit message: routed and filled
Parts:
- C307: value C11 -> 27n
- C308: value C9 -> 27n
- C309: value C10 -> 12n
- C311: value C12 -> 39n
- C312: value C8 -> 2n7
- C313: value C6 -> 33n
- C316: value C7 -> 15n
- C317: value C4 -> 33n
- D309, D310, D311, D313: footprint Diode_SMD:D_SOD-123 -> Diode_SMD:D_MiniMELF
- R324: value R17 -> 2k5
- R325: value R18 -> 6k8
- moved R307 103.9 mm to (115.0, 144.0), turned to 90 degrees
- moved R324 100.3 mm to (112.0, 69.5), turned to 180 degrees
- moved R303 95.7 mm to (108.5, 126.0), turned to 180 degrees
- moved R345 95.2 mm to (128.0, 144.0), turned to 90 degrees
- moved C309 94.5 mm to (135.0, 66.0), turned to 180 degrees
- moved R344 94.3 mm to (108.5, 124.0)
- moved C307 93.2 mm to (112.0, 71.5)
- moved R343 90.4 mm to (122.5, 125.0), turned to 180 degrees
- moved R301 90.4 mm to (114.5, 129.5)
- moved R336 88.9 mm to (112.5, 124.0), turned to 180 degrees
- moved R305 88.5 mm to (125.0, 144.0), turned to 90 degrees
- moved R337 87.2 mm to (122.5, 129.5), turned to 180 degrees
- moved R341 84.8 mm to (131.0, 135.0), turned to 270 degrees
- moved R342 83.7 mm to (126.5, 127.0), turned to 180 degrees
- moved R338 83.6 mm to (118.5, 129.5), turned to 180 degrees
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Connections:
- C315 pad 1: InGate -> InGate2
- D303 pad 1: NoiseIn -> NoiseIn2
- D304 pad 1: InAccent -> InAccent2
- D307 pad 1: InGate -> InGate2
- R301 pad 2: NoiseIn -> NoiseIn2
- R302 pad 2: InAccent -> InAccent2
- R303 pad 1: NoiseIn -> NoiseIn2
- R304 pad 1: InAccent -> InAccent2
- R305 pad 2: InGate -> InGate2
- R306 pad 1: InGate -> InGate2
- R307 pad 2: OutTom -> OutTom2
- R312 pad 1: InAccent -> InAccent2
- R314 pad 2: InAccent -> InAccent2
- R319 pad 2: OutTom -> OutTom2
- R326 pad 2: (no net) -> Net-(C312-Pad1)
- R331 pad 1: (no net) -> Net-(Q303-Pad1)
- R338 pad 2: NoiseIn -> NoiseIn2
- R345 pad 2: InGate -> InGate2
- TP301 pad 1: (no net) -> /KicadJE_AteOhAte3/Coupling
Routing:
- net GND: track 207.9 -> 332.3 mm, vias 78 -> 118
- net +12V: track 238.2 -> 356.1 mm, vias 0 -> 2
- net Net-(C308-Pad2): track 0.00 -> 90.0 mm, vias 0 -> 2
- net -12V: track 157.3 -> 239.6 mm, vias 0 -> 2
- net Net-(C317-Pad1): track 0.00 -> 81.0 mm, vias 0 -> 2
- net Net-(C313-Pad1): track 0.00 -> 74.3 mm
- net InAccent2: track 0.00 -> 67.9 mm, vias 0 -> 2
- net Net-(R311-Pad2): track 0.00 -> 65.0 mm, vias 0 -> 2
- net /KicadJE_AteOhAte3/Coupling: track 0.00 -> 60.1 mm, vias 0 -> 2
- net Net-(C310-Pad1): track 0.00 -> 50.2 mm, vias 0 -> 2
- net Net-(C311-Pad1): track 0.00 -> 41.4 mm
- net Net-(R341-Pad1): track 0.00 -> 38.2 mm, vias 0 -> 4
- net Net-(C310-Pad2): track 0.00 -> 37.7 mm, vias 0 -> 2
- net OutTom2: track 0.00 -> 35.5 mm, vias 0 -> 4
- net Net-(Q302-Pad1): track 0.00 -> 32.1 mm
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Other:
- board text added: "DRUM_Ate0Ate_Tom_1 Rev B - 04/10-2019 Johansen Engineering"
- board text added: "DRUM_Ate0Ate_Tom_2 Rev B - 04/10-2019 Johansen Engineering"
- board text removed: "DRUM_Ate0Ate_Tom_1 Rev A - 25/09-2019 Johansen Engineering"
