File: KicadJE_AteOhAte - RevB/KicadJE_AteOhAte3.sch (KiCad schematic (older format))
At the start: 120 parts

Commit message: New tom ext noise
Parts:
- removed C? (x4): 100n, Capacitor_SMD:C_0805_2012Metric_Pad1.15x1.40mm_HandSolder, symbol Device:C
- removed C?: 10n, Capacitor_SMD:C_0805_2012Metric_Pad1.15x1.40mm_HandSolder, symbol Device:C
- removed C?: C9, Capacitor_SMD:C_0805_2012Metric_Pad1.15x1.40mm_HandSolder, symbol Device:C
- removed C?: C10, Capacitor_SMD:C_0805_2012Metric_Pad1.15x1.40mm_HandSolder, symbol Device:C
- removed C?: C12, Capacitor_SMD:C_0805_2012Metric_Pad1.15x1.40mm_HandSolder, symbol Device:C
- removed C?: 10u, Capacitor_SMD:C_1206_3216Metric_Pad1.42x1.75mm_HandSolder, symbol Device:C
- removed C?: 22u, Capacitor_SMD:C_0805_2012Metric_Pad1.15x1.40mm_HandSolder, symbol Device:C
- removed C?: 1u, Capacitor_SMD:C_0805_2012Metric_Pad1.15x1.40mm_HandSolder, symbol Device:C
- removed C?: 39n, Capacitor_SMD:C_0805_2012Metric_Pad1.15x1.40mm_HandSolder, symbol Device:C
- removed C?: 18n, Capacitor_SMD:C_0805_2012Metric_Pad1.15x1.40mm_HandSolder, symbol Device:C
- removed D? (x2): D_Zener, Diode_SMD:D_MiniMELF, symbol Device:D_Zener
- removed J?: In_Accent, Connector_Audio:Jack_3.5mm_Ledino_KB3SPRS_Horizontal, symbol Connector:AudioJack2_SwitchT
- removed J?: In Gate, AJ-Dropbox-Kicad:PJ301SM, symbol Connector:AudioJack2_SwitchT
- removed J?: Out Tom, AJ-Dropbox-Kicad:PJ301SM, symbol Connector:AudioJack2
- removed JP?: Jumper, Connector_PinHeader_2.54mm:PinHeader_1x02_P2.54mm_Vertical, symbol Device:Jumper
- removed P?: Doepfer_Power_10pin, Connectors_IDC:IDC-Header_2x05_Pitch2.54mm_Straight, symbol Eurorack:Doepfer_Power_10pin
- removed Q? (x3): MMBT2222A, Package_TO_SOT_SMD:SOT-23_Handsoldering, symbol MMBT2222A:MMBT2222A
- removed R?: 1K, Resistor_SMD:R_0805_2012Metric_Pad1.15x1.40mm_HandSolder, symbol Device:R
- removed R?: OPEN, Resistor_SMD:R_0805_2012Metric_Pad1.15x1.40mm_HandSolder, symbol Device:R
- removed R?: 0R, Resistor_SMD:R_0805_2012Metric_Pad1.15x1.40mm_HandSolder, symbol Device:R
- removed R? (x5): 4k7, Resistor_SMD:R_0805_2012Metric_Pad1.15x1.40mm_HandSolder, symbol Device:R
- removed R?: 100k, Resistor_SMD:R_0805_2012Metric_Pad1.15x1.40mm_HandSolder, symbol Device:R
- removed R?: 15k, Resistor_SMD:R_0805_2012Metric_Pad1.15x1.40mm_HandSolder, symbol Device:R
- removed R? (x3): 10k, Resistor_SMD:R_0805_2012Metric_Pad1.15x1.40mm_HandSolder, symbol Device:R
- removed R? (x4): 22k, Resistor_SMD:R_0805_2012Metric_Pad1.15x1.40mm_HandSolder, symbol Device:R
- removed R? (x2): 33k, Resistor_SMD:R_0805_2012Metric_Pad1.15x1.40mm_HandSolder, symbol Device:R
- removed R?: 470k, Resistor_SMD:R_0805_2012Metric_Pad1.15x1.40mm_HandSolder, symbol Device:R
- removed R?: 1k, Resistor_SMD:R_0805_2012Metric_Pad1.15x1.40mm_HandSolder, symbol Device:R
- removed R?: 100R, Resistor_SMD:R_0805_2012Metric_Pad1.15x1.40mm_HandSolder, symbol Device:R
- removed R? (x2): 1M, Resistor_SMD:R_0805_2012Metric_Pad1.15x1.40mm_HandSolder, symbol Device:R
- removed R?: 300R, Resistor_SMD:R_0805_2012Metric_Pad1.15x1.40mm_HandSolder, symbol Device:R
- removed R?: 330K, Resistor_SMD:R_0805_2012Metric_Pad1.15x1.40mm_HandSolder, symbol Device:R
- removed RV?: 100K, Potentiometer_THT:Potentiometer_Bourns_3296W_Vertical, symbol Device:R_POT_TRIM
- removed RV?: 50K, Potentiometer_THT:Potentiometer_Bourns_3296W_Vertical, symbol Device:R_POT_TRIM
- removed SW? (x2): Con/Tom, AJ-Dropbox-Kicad:SPDTx2, symbol Switch:SW_DPDT_x2
- removed TP?: WhiteNoise, TestPoint:TestPoint_Pad_1.5x1.5mm, symbol Connector:TestPoint
- removed TP?: GND, TestPoint:TestPoint_THTPad_2.0x2.0mm_Drill1.0mm, symbol Connector:TestPoint
- removed U? (x4): TL072, AJ-Dropbox-Kicad:AJ_SO-8_5.3x6.2mm_P1.27mm, symbol Amplifier_Operational:TL072
- added C301: 10u, Capacitor_SMD:C_1206_3216Metric_Pad1.42x1.75mm_HandSolder, symbol Device:C
- added C302, C303, C305, C306: 100n, Capacitor_SMD:C_0805_2012Metric_Pad1.15x1.40mm_HandSolder, symbol Device:C
- added C308: C9, Capacitor_SMD:C_0805_2012Metric_Pad1.15x1.40mm_HandSolder, symbol Device:C
- added C309: C10, Capacitor_SMD:C_0805_2012Metric_Pad1.15x1.40mm_HandSolder, symbol Device:C
- added C311: C12, Capacitor_SMD:C_0805_2012Metric_Pad1.15x1.40mm_HandSolder, symbol Device:C
- added C315: 10n, Capacitor_SMD:C_0805_2012Metric_Pad1.15x1.40mm_HandSolder, symbol Device:C
- added D303, D304, D305, D306, D307, D308: Zener, Diode_SMD:D_MiniMELF, symbol Device:D_Zener
- added J301: Noise_In, Connector_Audio:Jack_3.5mm_Ledino_KB3SPRS_Horizontal, symbol Connector:AudioJack2_SwitchT
- added J302: In_Accent, Connector_Audio:Jack_3.5mm_Ledino_KB3SPRS_Horizontal, symbol Connector:AudioJack2_SwitchT
- added J303: In Gate, AJ-Dropbox-Kicad:PJ301SM, symbol Connector:AudioJack2_SwitchT
- added J304: Out Tom, AJ-Dropbox-Kicad:PJ301SM, symbol Connector:AudioJack2
- added P301: Doepfer_Power_10pin, Connectors_IDC:IDC-Header_2x05_Pitch2.54mm_Straight, symbol Eurorack:Doepfer_Power_10pin
- added Q302, Q305: MMBT2222A, Package_TO_SOT_SMD:SOT-23_Handsoldering, symbol MMBT2222A:MMBT2222A
- added R301, R305: 1K, Resistor_SMD:R_0805_2012Metric_Pad1.15x1.40mm_HandSolder, symbol Device:R
- added R303, R306: OPEN, Resistor_SMD:R_0805_2012Metric_Pad1.15x1.40mm_HandSolder, symbol Device:R
- added R307: 0R, Resistor_SMD:R_0805_2012Metric_Pad1.15x1.40mm_HandSolder, symbol Device:R
- added R309: 470k, Resistor_SMD:R_0805_2012Metric_Pad1.15x1.40mm_HandSolder, symbol Device:R
- added R311, R317: 33k, Resistor_SMD:R_0805_2012Metric_Pad1.15x1.40mm_HandSolder, symbol Device:R
- added R313: 100k, Resistor_SMD:R_0805_2012Metric_Pad1.15x1.40mm_HandSolder, symbol Device:R
- added R315, R323, R332, R336: 4k7, Resistor_SMD:R_0805_2012Metric_Pad1.15x1.40mm_HandSolder, symbol Device:R
- added R319: 1k, Resistor_SMD:R_0805_2012Metric_Pad1.15x1.40mm_HandSolder, symbol Device:R
- added R320: 15k, Resistor_SMD:R_0805_2012Metric_Pad1.15x1.40mm_HandSolder, symbol Device:R
- added R330, R331, R340: 10k, Resistor_SMD:R_0805_2012Metric_Pad1.15x1.40mm_HandSolder, symbol Device:R
- added R334, R335: 22k, Resistor_SMD:R_0805_2012Metric_Pad1.15x1.40mm_HandSolder, symbol Device:R
- added SW301: Con/Tom, AJ-Dropbox-Kicad:SPDTx2, symbol Switch:SW_DPDT_x2
- added unit 3 of U301
- added unit 2 of U302
- gave numbers to parts that had none: 59
Connections:
- net +12V: now also R313.2, R336.2
- net +12v: now also P301.10 (+12), P301.9 (+12), U301.4 (V-)
- net -12v: now also P301.1 (-12), P301.2 (-12), U301.8 (V+)
- net Coupling: now also R332.2
- net GND: now also D305.1 (K), D306.1 (K), D308.1 (K), J301.S, J301.TN, J302.S, J302.TN, J303.S, J303.TN, J304.S, P301.3 (GND), P301.4 (GND), P301.7 (GND), P301.8 (GND), Q305.2 (E), R303.2, R306.2, R331.2, R332.1, R340.1, SW301.4 (A)
- net InAccent: now also D304.1 (K)
- net InGate: now also C315.1, D307.1 (K), R305.2, R306.1
- net NoiseIn: now also D303.1 (K), R301.2, R303.1
- net OutTom: now also R307.2, R319.2
- net PNP_B: now also R323.1, R330.2
- net PNP_E: now also R323.2
- net at R302.1: now also J302.T
- net at C310.2, R316.1, RV303.2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: now also R319.1
- net at C310.1, R316.2, RV303.1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: now also C311.2
- net at U301.6 (-): now also R311.1, R317.2
- net at R318.1, RV302.2, U301.7: now also R311.2
- net at RV302.3: now also R309.1
- net at C307.2, R310.1, U301.1: now also C309.2, R317.1
- net at R310.2, U301.2 (-): now also C308.1
- net at R324.2: now also SW301.5 (B)
- net at C307.1: now also SW301.2 (B)
- net at D309.2 (A), D310.1 (K), R308.2: now also C308.2, C309.1, R309.2, SW301.3 (C)
- net at R341.1, R346.2: now also U302.5 (+)
- net at R347.2, R348.1: now also U302.6 (-)
- net at Q303.1 (B): now also R334.2
- net at Q303.3 (C): now also R320.1
- net at R314.1: now also Q302.3 (C), R315.2
- net at D313.1 (K), R341.2: now also C315.2
- net at Q301.1 (B): now also R313.1, R315.1
- net at R321.1, R329.2: now also Q302.2 (E)
- net at C313.2, Q306.3 (C): now also R336.1
- net at R318.2, R328.1: now also C311.1
- net at C304.2: now also C301.1
- new net: J301.T, R301.1
- new net: D303.2 (A), D306.2 (A)
- new net: D304.2 (A), D305.2 (A)
- new net: D307.2 (A), D308.2 (A)
- new net: C302.1, C305.2
- new net: J303.T, R305.1
- new net: J304.T, R307.1
- new net: C303.1, C306.2
- new net: R334.1, R335.2, U302.7
- new net: Q302.1 (B), R320.2
- new net: Q305.1 (B), R335.1, R340.2
- new net: Q305.3 (C), R330.1
Other:
- note removed: "Trim for 130mV RMS"

Commit message: Main components placed
Parts:
- removed U303: TL072, AJ-Dropbox-Kicad:AJ_SO-8_5.3x6.2mm_P1.27mm, symbol Amplifier_Operational:TL072
- J301: footprint Connector_Audio:Jack_3.5mm_Ledino_KB3SPRS_Horizontal -> AJ-Dropbox-Kicad:PJ301SM
Connections:
- net +12v is gone; now on net +12V: P301.10 (+12), P301.9 (+12), U301.4 (V-)
- net -12v is gone; now on net -12V: P301.1 (-12), P301.2 (-12), U301.8 (V+)
- net +12V: now also C304.1, C305.1, C306.1, D302.2 (A), U302.4 (V-)
- net -12V: now also C301.2, C302.2, C303.2, D301.1 (K), U302.8 (V+)
- net GND: now also C301.1, C302.1, C303.1, C304.2, C305.2, C306.2, D301.2 (A), D302.1 (K)
Changed lines of the file:
@@
-$EndComp
-$Comp
-L Amplifier_Operational:TL072 U303
-U 3 1 5D4ABFB1
-P 8825 1400
-F 0 "U303" H 8725 2150 50  0000 C CNN
-F 1 "TL072" H 8700 2000 50  0000 C CNN
-F 2 "AJ-Dropbox-Kicad:AJ_SO-8_5.3x6.2mm_P1.27mm" H 8825 1400 50  0001 C CNN
-F 3 "http://www.ti.com/lit/ds/symlink/tl071.pdf" H 8825 1400 50  0001 C CNN
-	3    8825 1400
-	1    0    0    -1
 $EndComp
 $Comp
@@
 	850  5500 850  6400
 Wire Wire Line
-	8525 1400 9900 1400
-Wire Wire Line
-	8550 1700 10050 1700
-Wire Wire Line
-	8550 1100 9850 1100
+	8525 1400 8950 1400
+Wire Wire Line
+	8550 1100 8650 1100
 Wire Wire Line
 	10600 2175 10450 2175
@@
 F 0 "J301" H 10567 2346 50  0000 R CNN
 F 1 "Noise_In" H 10567 2255 50  0000 R CNN
-F 2 "Connector_Audio:Jack_3.5mm_Ledino_KB3SPRS_Horizontal" H 10800 2275 50  0001 C CNN
+F 2 "AJ-Dropbox-Kicad:PJ301SM" H 10800 2275 50  0001 C CNN
 F 3 "~" H 10800 2275 50  0001 C CNN
 F 4 "VC input" H 10800 2275 50  0001 C CNN "Function"
@@
 Wire Wire Line
 	8275 2650 8400 2650
+Wire Wire Line
+	9850 1100 9800 1100
+Connection ~ 8650 1100
+Wire Wire Line
+	8650 1100 8950 1100
+Connection ~ 8950 1100
+Wire Wire Line
+	8950 1100 9175 1100
+Connection ~ 9175 1100
+Wire Wire Line
+	9175 1100 9400 1100
+Connection ~ 9400 1100
+Wire Wire Line
+	9400 1100 9600 1100
+Connection ~ 9600 1100
+Wire Wire Line
+	9600 1100 9800 1100
+Connection ~ 9800 1100
+Wire Wire Line
+	8550 1700 8650 1700
+Connection ~ 8650 1700
+Wire Wire Line
+	8650 1700 8950 1700
+Connection ~ 9800 1700
+Wire Wire Line
+	9800 1700 10050 1700
+Connection ~ 8950 1700
+Wire Wire Line
+	8950 1700 9175 1700
+Connection ~ 9175 1700
+Wire Wire Line
+	9175 1700 9400 1700
+Connection ~ 9400 1700
+Wire Wire Line
+	9400 1700 9600 1700
+Connection ~ 9600 1700
+Wire Wire Line
+	9600 1700 9800 1700
+Connection ~ 8950 1400
+Wire Wire Line
+	8950 1400 9175 1400
+Connection ~ 9175 1400
+Wire Wire Line
+	9175 1400 9400 1400
+Connection ~ 9400 1400
+Wire Wire Line
+	9400 1400 9600 1400
+Connection ~ 9600 1400
+Wire Wire Line
+	9600 1400 9900 1400
 $EndSCHEMATC

Commit message: Input placement
Parts:
- C307: value C11 -> 27n
- C308: value C9 -> 27n
- C309: value C10 -> 12n
- C311: value C12 -> 39n
- C312: value C8 -> 2n7
- C313: value C6 -> 33n
- C316: value C7 -> 15n
- C317: value C4 -> 33n
- R324: value R17 -> 2k5
- R325: value R18 -> 6k8
Connections:
- net InAccent renamed InAccent2
- net InGate renamed InGate2
- net NoiseIn renamed NoiseIn2
- net OutTom renamed OutTom2
Changed lines of the file:
@@
 $EndComp
 Text GLabel 1250 4900 0    50   Input ~ 0
-InAccent
+InAccent2
 Text GLabel 650  6700 1    50   Input ~ 0
-InGate
+InGate2
 $Comp
 L Device:R R314
@@
 P 4500 7100
 F 0 "C317" V 4400 7150 50  0000 L CNN
-F 1 "C4" H 4550 7000 50  0000 L CNN
+F 1 "33n" H 4550 7000 50  0000 L CNN
 F 2 "Capacitor_SMD:C_0805_2012Metric_Pad1.15x1.40mm_HandSolder" H 4538 6950 50  0001 C CNN
 F 3 "~" H 4500 7100 50  0001 C CNN
@@
 P 6050 6600
 F 0 "C313" V 5850 6525 50  0000 L CNN
-F 1 "C6" V 6200 6450 50  0000 L CNN
+F 1 "33n" V 6200 6450 50  0000 L CNN
 F 2 "Capacitor_SMD:C_0805_2012Metric_Pad1.15x1.40mm_HandSolder" H 6088 6450 50  0001 C CNN
 F 3 "~" H 6050 6600 50  0001 C CNN
@@
 P 4000 5750
 F 0 "C312" V 3900 5800 50  0000 L CNN
-F 1 "C8" H 4050 5650 50  0000 L CNN
+F 1 "2n7" H 4050 5650 50  0000 L CNN
 F 2 "Capacitor_SMD:C_0805_2012Metric_Pad1.15x1.40mm_HandSolder" H 4038 5600 50  0001 C CNN
 F 3 "~" H 4000 5750 50  0001 C CNN
@@
 P 4550 5350
 F 0 "R324" V 4550 5350 50  0000 C CNN
-F 1 "R17" V 4450 5425 50  0000 C CNN
+F 1 "2k5" V 4450 5425 50  0000 C CNN
 F 2 "Resistor_SMD:R_0805_2012Metric_Pad1.15x1.40mm_HandSolder" V 4480 5350 50  0001 C CNN
 F 3 "~" H 4550 5350 50  0001 C CNN
@@
 P 4850 5350
 F 0 "R325" V 4850 5350 50  0000 C CNN
-F 1 "R18" V 4750 5425 50  0000 C CNN
+F 1 "6k8" V 4750 5425 50  0000 C CNN
 F 2 "Resistor_SMD:R_0805_2012Metric_Pad1.15x1.40mm_HandSolder" V 4780 5350 50  0001 C CNN
 F 3 "~" H 4850 5350 50  0001 C CNN
@@
 P 4900 4300
 F 0 "C308" V 4700 4225 50  0000 L CNN
-F 1 "C9" V 5050 4150 50  0000 L CNN
+F 1 "27n" V 5050 4150 50  0000 L CNN
 F 2 "Capacitor_SMD:C_0805_2012Metric_Pad1.15x1.40mm_HandSolder" H 4938 4150 50  0001 C CNN
 F 3 "~" H 4900 4300 50  0001 C CNN
@@
 P 5400 4300
 F 0 "C309" V 5200 4225 50  0000 L CNN
-F 1 "C10" V 5450 4350 50  0000 L CNN
+F 1 "12n" V 5450 4350 50  0000 L CNN
 F 2 "Capacitor_SMD:C_0805_2012Metric_Pad1.15x1.40mm_HandSolder" H 5438 4150 50  0001 C CNN
 F 3 "~" H 5400 4300 50  0001 C CNN
@@
 P 5850 4100
 F 0 "C307" H 5750 4000 50  0000 L CNN
-F 1 "C11" H 5900 4200 50  0000 L CNN
+F 1 "27n" H 5900 4200 50  0000 L CNN
 F 2 "Capacitor_SMD:C_0805_2012Metric_Pad1.15x1.40mm_HandSolder" H 5888 3950 50  0001 C CNN
 F 3 "~" H 5850 4100 50  0001 C CNN
@@
 P 7600 5100
 F 0 "C311" V 7400 5025 50  0000 L CNN
-F 1 "C12" V 7650 5150 50  0000 L CNN
+F 1 "39n" V 7650 5150 50  0000 L CNN
 F 2 "Capacitor_SMD:C_0805_2012Metric_Pad1.15x1.40mm_HandSolder" H 7638 4950 50  0001 C CNN
 F 3 "~" H 7600 5100 50  0001 C CNN
@@
 P 6750 6900
 F 0 "C316" V 6650 6950 50  0000 L CNN
-F 1 "C7" H 6800 6800 50  0000 L CNN
+F 1 "15n" H 6800 6800 50  0000 L CNN
 F 2 "Capacitor_SMD:C_0805_2012Metric_Pad1.15x1.40mm_HandSolder" H 6788 6750 50  0001 C CNN
 F 3 "~" H 6750 6900 50  0001 C CNN
@@
 $EndComp
 Text GLabel 9050 5050 1    50   Input ~ 0
-OutTom
+OutTom2
 Wire Wire Line
 	9050 5200 9050 5050
@@
 $EndComp
 Text GLabel 7650 2300 0    50   Input ~ 0
-InAccent
+InAccent2
 Text GLabel 7650 2750 0    50   Input ~ 0
-InGate
+InGate2
 $Comp
 L Connector:AudioJack2 J304
@@
 	10450 3025 10450 2825
 Text GLabel 9950 2925 0    50   Input ~ 0
-OutTom
+OutTom2
 Wire Wire Line
 	7825 2600 7825 2650
@@
 Connection ~ 5100 6450
 Text GLabel 5500 6300 1    50   Input ~ 0
-NoiseIn
+NoiseIn2
 Wire Wire Line
 	5500 6300 5500 6450
@@
 	1    0    0    -1
 $EndComp
-Text GLabel 9700 2275 0    50   Input ~ 0
-NoiseIn
 Text Label 3300 5650 0    50   ~ 0
 PNP_B
@@
 Wire Wire Line
 	9600 1400 9900 1400
+Text GLabel 9700 2275 0    50   Input ~ 0
+NoiseIn2
 $EndSCHEMATC

Commit message: routed and filled
Parts:
- D309, D310, D311, D313: footprint Diode_SMD:D_SOD-123 -> Diode_SMD:D_MiniMELF
Connections:
- net Coupling: now also TP301.1
- net at Q303.1 (B), R334.2: now also R331.1
- net at C312.1, D311.1 (K): now also R326.2
Other:
- moved on the sheet: TP301
Changed lines of the file:
@@
 F 0 "D311" V 4425 6125 50  0000 L CNN
 F 1 "1N4148" V 4250 6100 50  0000 L CNN
-F 2 "Diode_SMD:D_SOD-123" H 4350 6200 50  0001 C CNN
+F 2 "Diode_SMD:D_MiniMELF" H 4350 6200 50  0001 C CNN
 F 3 "~" H 4350 6200 50  0001 C CNN
 	1    4350 6200
@@
 F 0 "D309" H 4950 3850 50  0000 L CNN
 F 1 "1N4148" V 4900 3900 50  0000 L CNN
-F 2 "Diode_SMD:D_SOD-123" H 4900 3800 50  0001 C CNN
+F 2 "Diode_SMD:D_MiniMELF" H 4900 3800 50  0001 C CNN
 F 3 "~" H 4900 3800 50  0001 C CNN
 	1    4900 3800
@@
 F 0 "D310" H 4650 3900 50  0000 L CNN
 F 1 "1N4148" V 5000 3650 50  0000 L CNN
-F 2 "Diode_SMD:D_SOD-123" H 4900 3950 50  0001 C CNN
+F 2 "Diode_SMD:D_MiniMELF" H 4900 3950 50  0001 C CNN
 F 3 "~" H 4900 3950 50  0001 C CNN
 	1    4900 3950
@@
 F 0 "D313" V 1050 7200 50  0000 L CNN
 F 1 "1N4148" V 950 7050 50  0000 L CNN
-F 2 "Diode_SMD:D_SOD-123" H 1050 7150 50  0001 C CNN
+F 2 "Diode_SMD:D_MiniMELF" H 1050 7150 50  0001 C CNN
 F 3 "~" H 1050 7150 50  0001 C CNN
 	1    1050 7150
@@
 L Connector:TestPoint TP301
 U 1 1 5DA7BFEF
-P 3800 5950
-F 0 "TP301" H 3858 6068 50  0000 L CNN
-F 1 "Coupling" H 3858 5977 50  0000 L CNN
-F 2 "TestPoint:TestPoint_Pad_1.5x1.5mm" H 4000 5950 50  0001 C CNN
-F 3 "~" H 4000 5950 50  0001 C CNN
-	1    3800 5950
+P 3825 5850
+F 0 "TP301" H 3883 5968 50  0000 L CNN
+F 1 "Coupling" H 3883 5877 50  0000 L CNN
+F 2 "TestPoint:TestPoint_Pad_1.5x1.5mm" H 4025 5850 50  0001 C CNN
+F 3 "~" H 4025 5850 50  0001 C CNN
+	1    3825 5850
 	1    0    0    -1
 $EndComp
@@
 	10750 1200 10750 1400
 Wire Wire Line
-	3650 5950 4000 5950
-Wire Wire Line
-	4000 5550 4350 5550
+	3650 5950 3825 5950
 Wire Wire Line
 	7650 2300 7825 2300
 Wire Wire Line
 	7650 2750 7825 2750
-Wire Wire Line
-	850  5500 850  6400
 Wire Wire Line
 	8525 1400 8950 1400
@@
 Text GLabel 9700 2275 0    50   Input ~ 0
 NoiseIn2
+Wire Wire Line
+	4000 5550 4100 5550
+Connection ~ 4100 5550
+Wire Wire Line
+	4100 5550 4350 5550
+Wire Wire Line
+	850  5500 850  6000
+Connection ~ 850  6000
+Wire Wire Line
+	850  6000 850  6400
+Wire Wire Line
+	3825 5850 3825 5950
+Connection ~ 3825 5950
+Wire Wire Line
+	3825 5950 4000 5950
 $EndSCHEMATC
